File: bcm-drum-synth.kicad_pcb (KiCad board)
At the start: 2 copper layers, 0 parts

Commit message: Rev 1
Parts:
- added C1: 47nF, Rumblesan_Footprints:C_Rect_L7.0mm_W3.5mm_P2.50mm_P5.00mm, F.Cu at (81.0, 46.7)
- added C10: 10uF, Capacitor_THT:CP_Radial_D5.0mm_P2.50mm, F.Cu at (112.1, 66.0)
- added C11: 47pF, Rumblesan_Footprints:C_Rect_L7.0mm_W3.5mm_P2.50mm_P5.00mm, F.Cu at (97.8, 75.7)
- added C12: 10uF, Capacitor_THT:CP_Radial_D5.0mm_P2.50mm, F.Cu at (117.3, 81.3)
- added C13: 1nF, Rumblesan_Footprints:C_Rect_L7.0mm_W3.5mm_P2.50mm_P5.00mm, F.Cu at (121.0, 54.9)
- added C14: 1nF, Rumblesan_Footprints:C_Rect_L7.0mm_W3.5mm_P2.50mm_P5.00mm, F.Cu at (152.5, 56.4)
- added C15: 1uF, Capacitor_THT:CP_Radial_D5.0mm_P2.50mm, F.Cu at (142.2, 91.9)
- added C16: 1nF, Rumblesan_Footprints:C_Rect_L7.0mm_W3.5mm_P2.50mm_P5.00mm, F.Cu at (145.7, 55.9)
- added C17: 1nF, Rumblesan_Footprints:C_Rect_L7.0mm_W3.5mm_P2.50mm_P5.00mm, F.Cu at (177.2, 57.9)
- added C18: 10uF, Capacitor_THT:CP_Radial_D5.0mm_P2.50mm, F.Cu at (183.0, 75.9)
- added C19: 100nF (X7R), Rumblesan_Footprints:C_Rect_L7.0mm_W3.5mm_P2.50mm_P5.00mm, F.Cu at (73.2, 68.6)
- added C2: 1uF, Capacitor_THT:CP_Radial_D5.0mm_P2.50mm, F.Cu at (95.5, 41.7)
- added C20: 1uF, Capacitor_THT:CP_Radial_D5.0mm_P2.50mm, F.Cu at (164.1, 38.2)
- added C21: 1uF, Capacitor_THT:CP_Radial_D5.0mm_P2.50mm, F.Cu at (172.2, 36.2)
- added C22: 100nF (X7R), Rumblesan_Footprints:C_Rect_L7.0mm_W3.5mm_P2.50mm_P5.00mm, F.Cu at (108.2, 65.0)
- added C23: 100nF (X7R), Rumblesan_Footprints:C_Rect_L7.0mm_W3.5mm_P2.50mm_P5.00mm, F.Cu at (96.5, 56.0)
- added C24: 100nF (X7R), Rumblesan_Footprints:C_Rect_L7.0mm_W3.5mm_P2.50mm_P5.00mm, F.Cu at (126.0, 58.9)
- added C25: 100nF (X7R), Rumblesan_Footprints:C_Rect_L7.0mm_W3.5mm_P2.50mm_P5.00mm, F.Cu at (145.7, 59.9)
- added C26: 100nF (X7R), Rumblesan_Footprints:C_Rect_L7.0mm_W3.5mm_P2.50mm_P5.00mm, F.Cu at (157.5, 60.5)
- added C27: 100nF (X7R), Rumblesan_Footprints:C_Rect_L7.0mm_W3.5mm_P2.50mm_P5.00mm, F.Cu at (177.2, 62.0)
- added C28: 100nF (X7R), Rumblesan_Footprints:C_Rect_L7.0mm_W3.5mm_P2.50mm_P5.00mm, F.Cu at (128.0, 97.0)
- added C29: 100nF (X7R), Rumblesan_Footprints:C_Rect_L7.0mm_W3.5mm_P2.50mm_P5.00mm, F.Cu at (124.8, 81.8)
- added C3: 47nF, Rumblesan_Footprints:C_Rect_L7.0mm_W3.5mm_P2.50mm_P5.00mm, F.Cu at (89.0, 48.8)
- added C30: 100nF (X7R), Rumblesan_Footprints:C_Rect_L7.0mm_W3.5mm_P2.50mm_P5.00mm, F.Cu at (165.6, 89.4)
- added C31: 100nF (X7R), Rumblesan_Footprints:C_Rect_L7.0mm_W3.5mm_P2.50mm_P5.00mm, F.Cu at (185.3, 88.9)
- added C4: 100nF, Rumblesan_Footprints:C_Rect_L7.0mm_W3.5mm_P2.50mm_P5.00mm, F.Cu at (68.1, 86.4)
- added C5: 100nF, Rumblesan_Footprints:C_Rect_L7.0mm_W3.5mm_P2.50mm_P5.00mm, F.Cu at (68.1, 82.3)
- added C6: 100nF, Rumblesan_Footprints:C_Rect_L7.0mm_W3.5mm_P2.50mm_P5.00mm, F.Cu at (73.0, 94.9)
- added C7: 47nF, Rumblesan_Footprints:C_Rect_L7.0mm_W3.5mm_P2.50mm_P5.00mm, F.Cu at (64.5, 60.5)
- added C8: 100nF, Rumblesan_Footprints:C_Rect_L7.0mm_W3.5mm_P2.50mm_P5.00mm, F.Cu at (53.3, 42.2)
- added C9: 100nF, Rumblesan_Footprints:C_Rect_L7.0mm_W3.5mm_P2.50mm_P5.00mm, F.Cu at (78.7, 70.6)
- added D1: D, Rumblesan_Footprints:Diode_THT_P7.62mm_Horizontal, F.Cu at (65.0, 86.4)
- added D10: LED, LED_THT:LED_D5.0mm, F.Cu at (185.5, 44.1)
- added D2: D, Rumblesan_Footprints:Diode_THT_P7.62mm_Horizontal, F.Cu at (65.0, 82.3)
- added D3: D, Rumblesan_Footprints:Diode_THT_P7.62mm_Horizontal, F.Cu at (68.1, 91.3)
- added D4: D, Rumblesan_Footprints:Diode_THT_P7.62mm_Horizontal, F.Cu at (117.3, 85.9)
- added D5: D, Rumblesan_Footprints:Diode_THT_P7.62mm_Horizontal, F.Cu at (132.1, 96.5)
- added D6: LED, LED_THT:LED_D5.0mm, F.Cu at (151.0, 91.9)
- added D7: 1N5189, Rumblesan_Footprints:D_DO-35_SOD27_P7.62mm_Horizontal, F.Cu at (160.0, 32.0)
- added D8: 1N5189, Rumblesan_Footprints:D_DO-35_SOD27_P7.62mm_Horizontal, F.Cu at (188.0, 35.8)
- added D9: LED, LED_THT:LED_D5.0mm, F.Cu at (157.1, 39.0)
- added J1: Input1, Connector_PinHeader_2.54mm:PinHeader_1x02_P2.54mm_Vertical, F.Cu at (53.8, 88.9)
- added J2: Input1, Connector_PinHeader_2.54mm:PinHeader_1x02_P2.54mm_Vertical, F.Cu at (53.8, 79.8)
- added J3: Trig_In, AudioJacks:Jack_3.5mm_QingPu_WQP-PJ398SM_Vertical, F.Cu at (58.5, 98.3)
- added J4: Freq_CV, AudioJacks:Jack_3.5mm_QingPu_WQP-PJ398SM_Vertical, F.Cu at (84.8, 113.0)
- added J5: Decay_CV, AudioJacks:Jack_3.5mm_QingPu_WQP-PJ398SM_Vertical, F.Cu at (143.8, 113.1)
- added J6: Audio_Out, AudioJacks:Jack_3.5mm_QingPu_WQP-PJ398SM_Vertical, F.Cu at (183.9, 112.9)
- added J7: Euro_Power, EurorackBasics:EurorackPowerHeader_2x05_P2.54mm_Shrouded, F.Cu at (173.1, 29.0)
- added Q1: 2N3904, Package_TO_SOT_THT:TO-92_Inline_Wide, F.Cu at (69.6, 60.5)
- added Q2: 2N3904, Package_TO_SOT_THT:TO-92_Inline_Wide, F.Cu at (58.4, 46.2)
- added Q3: 2N3904, Package_TO_SOT_THT:TO-92_Inline_Wide, F.Cu at (64.0, 71.0)
- added Q4: 2N3906, Package_TO_SOT_THT:TO-92_Inline_Wide, F.Cu at (99.1, 80.8)
- added Q5: 2N3906, Package_TO_SOT_THT:TO-92_Inline_Wide, F.Cu at (157.2, 101.7)
- added Q6: 2N3906, Package_TO_SOT_THT:TO-92_Inline_Wide, F.Cu at (151.9, 103.1)
- added R1: 22k, Resistor_THT:R_Axial_DIN0207_L6.3mm_D2.5mm_P7.62mm_Horizontal, F.Cu at (102.6, 42.2)
- added R10: R, Resistor_THT:R_Axial_DIN0207_L6.3mm_D2.5mm_P7.62mm_Horizontal, F.Cu at (64.5, 65.0)
- added R11: 100k, Resistor_THT:R_Axial_DIN0207_L6.3mm_D2.5mm_P7.62mm_Horizontal, F.Cu at (88.9, 42.2)
- added R12: 100k, Resistor_THT:R_Axial_DIN0207_L6.3mm_D2.5mm_P7.62mm_Horizontal, F.Cu at (110.2, 48.3)
- added R13: 100k, Resistor_THT:R_Axial_DIN0207_L6.3mm_D2.5mm_P7.62mm_Horizontal, F.Cu at (87.4, 92.5)
- added R14: 100k, Resistor_THT:R_Axial_DIN0207_L6.3mm_D2.5mm_P7.62mm_Horizontal, F.Cu at (65.5, 42.2)
- added R15: R, Resistor_THT:R_Axial_DIN0207_L6.3mm_D2.5mm_P7.62mm_Horizontal, F.Cu at (88.4, 66.5)
- added R16: 100k, Resistor_THT:R_Axial_DIN0207_L6.3mm_D2.5mm_P7.62mm_Horizontal, F.Cu at (102.6, 51.3)
- added R17: 100k, Resistor_THT:R_Axial_DIN0207_L6.3mm_D2.5mm_P7.62mm_Horizontal, F.Cu at (90.4, 92.5)
- added R18: 100k, Resistor_THT:R_Axial_DIN0207_L6.3mm_D2.5mm_P7.62mm_Horizontal, F.Cu at (81.0, 82.0)
- added R19: 100k, Resistor_THT:R_Axial_DIN0207_L6.3mm_D2.5mm_P7.62mm_Horizontal, F.Cu at (97.0, 84.8)
- added R2: 22k, Resistor_THT:R_Axial_DIN0207_L6.3mm_D2.5mm_P7.62mm_Horizontal, F.Cu at (73.2, 45.2)
- added R20: 15k, Resistor_THT:R_Axial_DIN0207_L6.3mm_D2.5mm_P7.62mm_Horizontal, F.Cu at (134.1, 110.2)
- added R21: 120k, Resistor_THT:R_Axial_DIN0207_L6.3mm_D2.5mm_P7.62mm_Horizontal, F.Cu at (138.7, 96.5)
- added R22: 100k, Resistor_THT:R_Axial_DIN0207_L6.3mm_D2.5mm_P7.62mm_Horizontal, F.Cu at (141.7, 104.1)
- added R23: 100k, Resistor_THT:R_Axial_DIN0207_L6.3mm_D2.5mm_P7.62mm_Horizontal, F.Cu at (110.7, 74.7)
- added R24: 100k, Resistor_THT:R_Axial_DIN0207_L6.3mm_D2.5mm_P7.62mm_Horizontal, F.Cu at (136.1, 78.2)
- added R25: R, Resistor_THT:R_Axial_DIN0207_L6.3mm_D2.5mm_P7.62mm_Horizontal, F.Cu at (113.8, 85.9)
- added R26: 220r, Resistor_THT:R_Axial_DIN0207_L6.3mm_D2.5mm_P7.62mm_Horizontal, F.Cu at (118.9, 65.5)
- added R27: 220r, Resistor_THT:R_Axial_DIN0207_L6.3mm_D2.5mm_P7.62mm_Horizontal, F.Cu at (158.0, 67.1)
- added R28: 220r, Resistor_THT:R_Axial_DIN0207_L6.3mm_D2.5mm_P7.62mm_Horizontal, F.Cu at (126.5, 68.6)
- added R29: 220r, Resistor_THT:R_Axial_DIN0207_L6.3mm_D2.5mm_P7.62mm_Horizontal, F.Cu at (158.0, 70.1)
- added R3: 100k, Resistor_THT:R_Axial_DIN0207_L6.3mm_D2.5mm_P7.62mm_Horizontal, F.Cu at (52.8, 63.0)
- added R30: 27k, Resistor_THT:R_Axial_DIN0207_L6.3mm_D2.5mm_P7.62mm_Horizontal, F.Cu at (133.6, 82.3)
- added R31: 100k, Resistor_THT:R_Axial_DIN0207_L6.3mm_D2.5mm_P7.62mm_Horizontal, F.Cu at (126.5, 62.5)
- added R32: 100k, Resistor_THT:R_Axial_DIN0207_L6.3mm_D2.5mm_P7.62mm_Horizontal, F.Cu at (158.0, 64.0)
- added R33: 100k, Resistor_THT:R_Axial_DIN0207_L6.3mm_D2.5mm_P7.62mm_Horizontal, F.Cu at (93.5, 84.8)
- added R34: 470r, Resistor_THT:R_Axial_DIN0207_L6.3mm_D2.5mm_P7.62mm_Horizontal, F.Cu at (158.0, 93.5)
- added R35: 4k3, Resistor_THT:R_Axial_DIN0207_L6.3mm_D2.5mm_P7.62mm_Horizontal, F.Cu at (147.4, 84.3)
- added R36: 470r, Resistor_THT:R_Axial_DIN0207_L6.3mm_D2.5mm_P7.62mm_Horizontal, F.Cu at (158.0, 96.6)
- added R37: 100k, Resistor_THT:R_Axial_DIN0207_L6.3mm_D2.5mm_P7.62mm_Horizontal, F.Cu at (158.0, 84.3)
- added R38: 10k, Resistor_THT:R_Axial_DIN0207_L6.3mm_D2.5mm_P7.62mm_Horizontal, F.Cu at (129.5, 50.3)
- added R39: 10k, Resistor_THT:R_Axial_DIN0207_L6.3mm_D2.5mm_P7.62mm_Horizontal, F.Cu at (161.0, 49.8)
- added R4: 100r, Resistor_THT:R_Axial_DIN0207_L6.3mm_D2.5mm_P7.62mm_Horizontal, F.Cu at (73.2, 48.3)
- added R40: 100k, Resistor_THT:R_Axial_DIN0207_L6.3mm_D2.5mm_P7.62mm_Horizontal, F.Cu at (129.5, 47.2)
- added R41: 100k, Resistor_THT:R_Axial_DIN0207_L6.3mm_D2.5mm_P7.62mm_Horizontal, F.Cu at (161.0, 52.8)
- added R42: 220r, Resistor_THT:R_Axial_DIN0207_L6.3mm_D2.5mm_P7.62mm_Horizontal, F.Cu at (140.2, 66.5)
- added R43: 220r, Resistor_THT:R_Axial_DIN0207_L6.3mm_D2.5mm_P7.62mm_Horizontal, F.Cu at (171.7, 68.6)
- added R44: R, Resistor_THT:R_Axial_DIN0207_L6.3mm_D2.5mm_P7.62mm_Horizontal, F.Cu at (124.0, 96.5)
- added R45: 220r, Resistor_THT:R_Axial_DIN0207_L6.3mm_D2.5mm_P7.62mm_Horizontal, F.Cu at (140.2, 69.6)
- added R46: 220r, Resistor_THT:R_Axial_DIN0207_L6.3mm_D2.5mm_P7.62mm_Horizontal, F.Cu at (171.7, 71.6)
- added R47: 220r, Resistor_THT:R_Axial_DIN0207_L6.3mm_D2.5mm_P7.62mm_Horizontal, F.Cu at (179.5, 95.6)
- added R48: 220r, Resistor_THT:R_Axial_DIN0207_L6.3mm_D2.5mm_P7.62mm_Horizontal, F.Cu at (179.5, 98.7)
- added R49: 100k, Resistor_THT:R_Axial_DIN0207_L6.3mm_D2.5mm_P7.62mm_Horizontal, F.Cu at (140.2, 63.5)
- added R5: 100r, Resistor_THT:R_Axial_DIN0207_L6.3mm_D2.5mm_P7.62mm_Horizontal, F.Cu at (102.6, 45.2)
- added R50: 100k, Resistor_THT:R_Axial_DIN0207_L6.3mm_D2.5mm_P7.62mm_Horizontal, F.Cu at (171.7, 65.5)
- added R51: 100k, Resistor_THT:R_Axial_DIN0207_L6.3mm_D2.5mm_P7.62mm_Horizontal, F.Cu at (187.1, 92.6)
- added R52: 10k, Resistor_THT:R_Axial_DIN0207_L6.3mm_D2.5mm_P7.62mm_Horizontal, F.Cu at (179.5, 85.2)
- added R53: R, Resistor_THT:R_Axial_DIN0207_L6.3mm_D2.5mm_P7.62mm_Horizontal, F.Cu at (144.8, 104.1)
- added R54: 10k, Resistor_THT:R_Axial_DIN0207_L6.3mm_D2.5mm_P7.62mm_Horizontal, F.Cu at (140.5, 51.9)
- added R55: 10k, Resistor_THT:R_Axial_DIN0207_L6.3mm_D2.5mm_P7.62mm_Horizontal, F.Cu at (172.2, 54.4)
- added R56: R, Resistor_THT:R_Axial_DIN0207_L6.3mm_D2.5mm_P7.62mm_Horizontal, F.Cu at (135.6, 96.5)
- added R57: 100k, Resistor_THT:R_Axial_DIN0207_L6.3mm_D2.5mm_P7.62mm_Horizontal, F.Cu at (150.4, 73.2)
- added R58: 10k, Resistor_THT:R_Axial_DIN0207_L6.3mm_D2.5mm_P7.62mm_Horizontal, F.Cu at (183.0, 80.6)
- added R59: 10k, Resistor_THT:R_Axial_DIN0207_L6.3mm_D2.5mm_P7.62mm_Horizontal, F.Cu at (168.7, 45.2)
- added R6: 1m, Resistor_THT:R_Axial_DIN0207_L6.3mm_D2.5mm_P7.62mm_Horizontal, F.Cu at (52.8, 59.9)
- added R60: 1k, Resistor_THT:R_Axial_DIN0207_L6.3mm_D2.5mm_P7.62mm_Horizontal, F.Cu at (151.0, 38.5)
- added R61: 6k8, Resistor_THT:R_Axial_DIN0207_L6.3mm_D2.5mm_P7.62mm_Horizontal, F.Cu at (125.5, 49.8)
- added R62: 1k, Resistor_THT:R_Axial_DIN0207_L6.3mm_D2.5mm_P7.62mm_Horizontal, F.Cu at (176.8, 115.8)
- added R63: 3k3, Resistor_THT:R_Axial_DIN0207_L6.3mm_D2.5mm_P7.62mm_Horizontal, F.Cu at (157.1, 24.3)
- added R64: 3k3, Resistor_THT:R_Axial_DIN0207_L6.3mm_D2.5mm_P7.62mm_Horizontal, F.Cu at (188.0, 38.7)
- added R7: 100k, Resistor_THT:R_Axial_DIN0207_L6.3mm_D2.5mm_P7.62mm_Horizontal, F.Cu at (60.5, 53.8)
- added R8: 6k8, Resistor_THT:R_Axial_DIN0207_L6.3mm_D2.5mm_P7.62mm_Horizontal, F.Cu at (60.5, 56.9)
- added R9: 22r, Resistor_THT:R_Axial_DIN0207_L6.3mm_D2.5mm_P7.62mm_Horizontal, F.Cu at (60.5, 50.8)
- added RV1: 1mA, Rumblesan_Footprints:Potentiometer_Alpha_RD901F-40-00D_Single_Vertical_CircularHoles, F.Cu at (108.7, 31.0)
- added RV10: 100k, Rumblesan_Footprints:Potentiometer_Alpha_RD901F-40-00D_Single_Vertical_CircularHoles, F.Cu at (97.0, 111.8)
- added RV11: 50kA, Rumblesan_Footprints:Potentiometer_Alpha_RD901F-40-00D_Single_Vertical_CircularHoles, F.Cu at (142.5, 31.0)
- added RV12: 100kA, Rumblesan_Footprints:Potentiometer_Alpha_RD901F-40-00D_Single_Vertical_CircularHoles, F.Cu at (167.6, 111.0)
- added RV2: 1mA, Rumblesan_Footprints:Potentiometer_Alpha_RD901F-40-00D_Single_Vertical_CircularHoles, F.Cu at (72.6, 31.0)
- added RV3: 100kA, Rumblesan_Footprints:Potentiometer_Alpha_RD901F-40-00D_Single_Vertical_CircularHoles, F.Cu at (86.9, 31.0)
- added RV4: 100kA, Rumblesan_Footprints:Potentiometer_Alpha_RD901F-40-00D_Single_Vertical_CircularHoles, F.Cu at (122.9, 31.0)
- added RV5: 100kB, Rumblesan_Footprints:Potentiometer_Alpha_RD901F-40-00D_Single_Vertical_CircularHoles, F.Cu at (72.6, 111.8)
- added RV6: 100kA, Rumblesan_Footprints:Potentiometer_Alpha_RD901F-40-00D_Single_Vertical_CircularHoles, F.Cu at (58.4, 31.0)
- added RV7: 100kB, Rumblesan_Footprints:Potentiometer_Alpha_RD901F-40-00D_Single_Vertical_CircularHoles, F.Cu at (58.4, 111.8)
- added RV8: 100k, Rumblesan_Footprints:Potentiometer_Alpha_RD901F-40-00D_Single_Vertical_CircularHoles, F.Cu at (125.5, 111.8)
- added RV9: 100k, Rumblesan_Footprints:Potentiometer_Alpha_RD901F-40-00D_Single_Vertical_CircularHoles, F.Cu at (111.3, 111.8)
- added SW1: SW_SPDT, Rumblesan_Footprints:SW_SPDT_DailyWell_MiniToggle, F.Cu at (98.0, 37.3)
- added TP1: TestPoint, TestPoint:TestPoint_Loop_D2.50mm_Drill1.0mm_LowProfile, F.Cu at (66.5, 76.6)
- added TP10: TestPoint, TestPoint:TestPoint_Loop_D2.50mm_Drill1.0mm_LowProfile, F.Cu at (183.5, 58.0)
- added TP11: TestPoint, TestPoint:TestPoint_Loop_D2.50mm_Drill1.0mm_LowProfile, F.Cu at (185.4, 68.5)
- added TP2: TestPoint, TestPoint:TestPoint_Loop_D2.50mm_Drill1.0mm_LowProfile, F.Cu at (115.1, 42.5)
- added TP3: TestPoint, TestPoint:TestPoint_Loop_D2.50mm_Drill1.0mm_LowProfile, F.Cu at (79.2, 23.9)
- added TP4: TestPoint, TestPoint:TestPoint_Loop_D2.50mm_Drill1.0mm_LowProfile, F.Cu at (52.6, 23.7)
- added TP5: TestPoint, TestPoint:TestPoint_Loop_D2.50mm_Drill1.0mm_LowProfile, F.Cu at (118.2, 98.6)
- added TP6: TestPoint, TestPoint:TestPoint_Loop_D2.50mm_Drill1.0mm_LowProfile, F.Cu at (114.7, 60.1)
- added TP7: TestPoint, TestPoint:TestPoint_Loop_D2.50mm_Drill1.0mm_LowProfile, F.Cu at (108.7, 80.8)
- added TP8: TestPoint, TestPoint:TestPoint_Loop_D2.50mm_Drill1.0mm_LowProfile, F.Cu at (97.4, 102.5)
- added TP9: TestPoint, TestPoint:TestPoint_Loop_D2.50mm_Drill1.0mm_LowProfile, F.Cu at (149.0, 99.1)
- added U1: HEF4093B, Package_DIP:DIP-14_W7.62mm_LongPads, F.Cu at (84.8, 66.5)
- added U2: TL072, Package_DIP:DIP-8_W7.62mm_LongPads, F.Cu at (104.1, 64.0)
- added U3: TL074, Package_DIP:DIP-14_W7.62mm_LongPads, F.Cu at (120.9, 93.5)
- added U4: LM13700, Package_DIP:DIP-16_W7.62mm_LongPads, F.Cu at (137.2, 71.1)
- added U5: LM13700, Package_DIP:DIP-16_W7.62mm_LongPads, F.Cu at (168.7, 74.2)
- added U6: LM13700, Package_DIP:DIP-16_W7.62mm_LongPads, F.Cu at (176.3, 102.1)
Routing:
- net +12V: track 0.00 -> 411.3 mm
- net -12V: track 0.00 -> 212.2 mm
- net Net-(C3-Pad2): track 0.00 -> 110.8 mm, vias 0 -> 1
- net Net-(R47-Pad1): track 0.00 -> 78.1 mm
- net Net-(C9-Pad2): track 0.00 -> 74.7 mm, vias 0 -> 1
- net Net-(C18-Pad2): track 0.00 -> 64.6 mm
- net /I_FREQ: track 0.00 -> 54.7 mm
- net Net-(RV10-Pad3): track 0.00 -> 49.4 mm
- net Net-(R11-Pad2): track 0.00 -> 48.2 mm
- net Net-(C15-Pad1): track 0.00 -> 47.4 mm
- net Net-(R18-Pad1): track 0.00 -> 46.6 mm
- net Net-(R4-Pad2): track 0.00 -> 41.2 mm
- net Net-(R20-Pad1): track 0.00 -> 34.5 mm
- net Net-(R49-Pad2): track 0.00 -> 33.9 mm
- net Net-(R26-Pad1): track 0.00 -> 33.5 mm
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- added copper zone on B.Cu, net GND
- added copper zone on F.Cu, net GND
Other:
- board outline added: 143.8 x 103.8 mm
- net class Default removed
- net class Power removed
- net class Signal removed
- board text added: "Filter Env Decay"
- board text added: "Filter Freq"
- board text added: "Filter LFO Mod"
- board text added: "Freq CV"
- board text added: "Freq Env"
- board text added: "Magnum Percussion Instrument rev 01"
- board text added: "Noise Level"
- board text added: "OSC1 Freq"
- board text added: "OSC1 Level"
- board text added: "OSC2 Freq"
- board text added: "OSC2 LFO"
- board text added: "OSC2 Level"
- board text added: "Out"
- board text added: "Output Volume"
- board text added: "Resonance"
- board text added: "Trig"
- board text added: "Volume Env CV"
- board text added: "Volume Env Decay"
