File: bcm-drum-synth.kicad_sch (KiCad schematic)
At the start: 88 parts

Commit message: Adding some info to schematic
Parts:
- removed C? (x2): 2uF, symbol Device:C_Polarized
- removed Q? (x5): 2N3904, Package_TO_SOT_THT:TO-92_Inline, symbol Transistor_BJT:2N3904
- removed R? (x2): R, symbol Device:R
- removed RV?: R_Potentiometer, symbol Device:R_Potentiometer
- added C? (x2): C, symbol Device:C
- added C? (x2): C_Polarized, symbol Device:C_Polarized
- added D? (x3): D, symbol Device:D
- added J? (x2): Input1, symbol Connector:Conn_01x02_Female
- added J? (x2): AudioJack2_SwitchT, symbol Connector:AudioJack2_SwitchT
- added Q?: 2N3904, Package_TO_SOT_THT:TO-92_Inline, symbol Transistor_BJT:2N3904
- added R?: 100r, symbol Device:R
- added R? (x11): R, symbol Device:R
- added RV? (x2): R_Potentiometer, symbol Device:R_Potentiometer
- added U? (x5): TL072, symbol Amplifier_Operational:TL072
Connections:
- net GND: now also C?.2, C?.2, J?.1 (Pin_1), J?.1 (Pin_1), J?.S, J?.S, Q?.1 (E), R?.1, R?.1, R?.2, RV?.1, RV?.2, RV?.3
- net +12V: now reaches R?.1
- net +12V: now also R?.1, R?.1, R?.1, R?.2, RV?.3
- net -12V: now reaches C?.2
- net -12V: now also C?.1, C?.1, Q?.2 (B), R?.2, R?.2, R?.2, R?.2, R?.2, R?.2
- net at U?.7: now also U?.5
- net at U?.8: now also R?.2
- net at RV?.1, RV?.2, RV?.3: now also R?.2; no longer U?.3
- net at R?.1, U?.1, U?.2: now also C?.2; no longer C?.1
- net at U?.3 (+): now also R?.2
- net at U?.4 (-): now also R?.1, R?.2
- net at U?.10: now also U?.13
- net at U?.8: now also U?.9, C?.2, R?.1
- net at U?.11: now also C?.1
- net at U?.12: now also Q?.3 (C), R?.2
- net at U?.5 (+): now also C?.1, D?.1 (K)
- net at U?.6 (-): now also U?.7
- new net: R?.1, U?.3
- new net: D?.2 (A), J?.2 (Pin_2), J?.2 (Pin_2), J?.T
- new net: R?.1, RV?.1
- new net: C?.1, D?.1 (K), R?.2, U?.5 (+)
- new net: D?.2 (A), U?.1, U?.2 (-)
- new net: R?.1, RV?.2
- new net: C?.1, D?.1 (K)
- new net: C?.2, Q?.2 (B)
- new net: J?.T, R?.1
- new net: D?.2 (A), R?.2
- new net: U?.6 (-), U?.7
- no-connect marks 6 -> 8
Other:
- note added: "Filter"
- note added: "Input Handling"
- note added: "LFO/OSC select"
- note added: "Mixer"
- note added: "Noise Level"
- note added: "Non Voltage Controlled Envelope"
- note added: "OSC1 Level"
- note added: "OSC2 Level"
- note added: "Output VCA"
- note added: "Power connections"
- moved on the sheet: C?, Q?, R?, RV?, SW?, U?A, U?B, U?C, U?D, U?E

Commit message: Rev 1
Parts:
- removed C?: C_Polarized, symbol Device:C_Polarized
- removed D?: D, symbol Device:D
- removed R?: R, symbol Device:R
- removed R?: 100k, symbol Device:R
- removed RV?: R_Potentiometer, symbol Device:R_Potentiometer
- removed SW?: SW_SPST, symbol Switch:SW_SPST
- removed U? (x5): TL072, symbol Amplifier_Operational:TL072
- added C10, C12, C18: 10uF, Capacitor_THT:CP_Radial_D5.0mm_P2.50mm, symbol Device:C_Polarized
- added C11: 47pF, Rumblesan_Footprints:C_Rect_L7.0mm_W3.5mm_P2.50mm_P5.00mm, symbol Device:C
- added C19, C22, C23, C24, C25, C26, C27, C28, C29, C30, C31: 100nF (X7R), Rumblesan_Footprints:C_Rect_L7.0mm_W3.5mm_P2.50mm_P5.00mm, symbol Device:C
- added C20, C21: 1uF, Capacitor_THT:CP_Radial_D5.0mm_P2.50mm, symbol Device:C_Polarized
- added C4, C5: 100nF, Rumblesan_Footprints:C_Rect_L7.0mm_W3.5mm_P2.50mm_P5.00mm, symbol Device:C
- added D1, D2, D4: D, Rumblesan_Footprints:Diode_THT_P7.62mm_Horizontal, symbol Device:D
- added D10, D6, D9: LED, LED_THT:LED_D5.0mm, symbol Device:LED
- added D7, D8: 1N5189, Rumblesan_Footprints:D_DO-35_SOD27_P7.62mm_Horizontal, symbol Device:D
- added J4: Freq_CV, AudioJacks:Jack_3.5mm_QingPu_WQP-PJ398SM_Vertical, symbol Connector:AudioJack2_SwitchT
- added J6: Audio_Out, AudioJacks:Jack_3.5mm_QingPu_WQP-PJ398SM_Vertical, symbol Connector:AudioJack2_SwitchT
- added J7: Euro_Power, EurorackBasics:EurorackPowerHeader_2x05_P2.54mm_Shrouded, symbol Connector_Generic:Conn_02x05_Odd_Even
- added Q4, Q5, Q6: 2N3906, Package_TO_SOT_THT:TO-92_Inline_Wide, symbol Transistor_BJT:2N3906
- added R13, R17, R18, R19, R23, R33: 100k, Resistor_THT:R_Axial_DIN0207_L6.3mm_D2.5mm_P7.62mm_Horizontal, symbol Device:R
- added R25, R53, R56: R, Resistor_THT:R_Axial_DIN0207_L6.3mm_D2.5mm_P7.62mm_Horizontal, symbol Device:R
- added R30: 27k, Resistor_THT:R_Axial_DIN0207_L6.3mm_D2.5mm_P7.62mm_Horizontal, symbol Device:R
- added R35: 4k3, Resistor_THT:R_Axial_DIN0207_L6.3mm_D2.5mm_P7.62mm_Horizontal, symbol Device:R
- added R59: 10k, Resistor_THT:R_Axial_DIN0207_L6.3mm_D2.5mm_P7.62mm_Horizontal, symbol Device:R
- added R60: 1k, Resistor_THT:R_Axial_DIN0207_L6.3mm_D2.5mm_P7.62mm_Horizontal, symbol Device:R
- added R61: 6k8, Resistor_THT:R_Axial_DIN0207_L6.3mm_D2.5mm_P7.62mm_Horizontal, symbol Device:R
- added R63, R64: 3k3, Resistor_THT:R_Axial_DIN0207_L6.3mm_D2.5mm_P7.62mm_Horizontal, symbol Device:R
- added RV10, RV9: 100k, Rumblesan_Footprints:Potentiometer_Alpha_RD901F-40-00D_Single_Vertical_CircularHoles, symbol Device:R_Potentiometer
- added RV11: 50kA, Rumblesan_Footprints:Potentiometer_Alpha_RD901F-40-00D_Single_Vertical_CircularHoles, symbol Device:R_Potentiometer
- added RV12: 100kA, Rumblesan_Footprints:Potentiometer_Alpha_RD901F-40-00D_Single_Vertical_CircularHoles, symbol Device:R_Potentiometer
- added RV5, RV7: 100kB, Rumblesan_Footprints:Potentiometer_Alpha_RD901F-40-00D_Single_Vertical_CircularHoles, symbol Device:R_Potentiometer
- added SW1: SW_SPDT, Rumblesan_Footprints:SW_SPDT_DailyWell_MiniToggle, symbol Switch:SW_SPDT
- added TP1, TP10, TP11, TP2, TP3, TP4, TP5, TP6, TP7, TP8, TP9: TestPoint, TestPoint:TestPoint_Loop_D2.50mm_Drill1.0mm_LowProfile, symbol Connector:TestPoint
- added U3: TL074, Package_DIP:DIP-14_W7.62mm_LongPads, symbol Amplifier_Operational:TL074
- C1, C13, C14, C16, C17, C3, C7, C8: renamed from C?; footprint (none) -> Rumblesan_Footprints:C_Rect_L7.0mm_W3.5mm_P2.50mm_P5.00mm
- C15: renamed from C?; value C_Polarized -> 1uF; footprint (none) -> Capacitor_THT:CP_Radial_D5.0mm_P2.50mm
- C2: renamed from C?; footprint (none) -> Capacitor_THT:CP_Radial_D5.0mm_P2.50mm
- C6, C9: renamed from C?; value C -> 100nF; footprint (none) -> Rumblesan_Footprints:C_Rect_L7.0mm_W3.5mm_P2.50mm_P5.00mm
- D3, D5: renamed from D?; footprint (none) -> Rumblesan_Footprints:Diode_THT_P7.62mm_Horizontal
- J1, J2: renamed from J?; footprint (none) -> Connector_PinHeader_2.54mm:PinHeader_1x02_P2.54mm_Vertical
- J3: renamed from J?; value AudioJack2_SwitchT -> Trig_In; footprint (none) -> AudioJacks:Jack_3.5mm_QingPu_WQP-PJ398SM_Vertical
- J5: renamed from J?; value AudioJack2_SwitchT -> Decay_CV; footprint (none) -> AudioJacks:Jack_3.5mm_QingPu_WQP-PJ398SM_Vertical
- Q1, Q2, Q3: renamed from Q?; footprint Package_TO_SOT_THT:TO-92_Inline -> Package_TO_SOT_THT:TO-92_Inline_Wide
- R1, R10, R11, R12, R14, R15, R16, R2, R26, R27, R28, R29, R3, R31, R32, R38, R39, R4, R40, R41, R42, R43, R44, R45, R46, R47, R48, R49, R5, R50, R51, R52, R54, R55, R57, R58, R6, R7, R8, R9: renamed from R?; footprint (none) -> Resistor_THT:R_Axial_DIN0207_L6.3mm_D2.5mm_P7.62mm_Horizontal
- R20: renamed from R?; value R -> 15k; footprint (none) -> Resistor_THT:R_Axial_DIN0207_L6.3mm_D2.5mm_P7.62mm_Horizontal
- R21: renamed from R?; value R -> 120k; footprint (none) -> Resistor_THT:R_Axial_DIN0207_L6.3mm_D2.5mm_P7.62mm_Horizontal
- R22, R24, R37: renamed from R?; value R -> 100k; footprint (none) -> Resistor_THT:R_Axial_DIN0207_L6.3mm_D2.5mm_P7.62mm_Horizontal
- R34, R36: renamed from R?; value R -> 470r; footprint (none) -> Resistor_THT:R_Axial_DIN0207_L6.3mm_D2.5mm_P7.62mm_Horizontal
- R62: renamed from R?; value 100k -> 1k; footprint (none) -> Resistor_THT:R_Axial_DIN0207_L6.3mm_D2.5mm_P7.62mm_Horizontal
- RV1, RV2, RV3, RV4, RV6: renamed from RV?; footprint (none) -> Rumblesan_Footprints:Potentiometer_Alpha_RD901F-40-00D_Single_Vertical_CircularHoles
- RV8: renamed from RV?; value R_Potentiometer -> 100k; footprint (none) -> Rumblesan_Footprints:Potentiometer_Alpha_RD901F-40-00D_Single_Vertical_CircularHoles
- U1: renamed from U?; footprint (none) -> Package_DIP:DIP-14_W7.62mm_LongPads
- U2: renamed from U?; footprint (none) -> Package_DIP:DIP-8_W7.62mm_LongPads
- U4, U5, U6: renamed from U?; footprint (none) -> Package_DIP:DIP-16_W7.62mm_LongPads
Connections:
- net +12V: now also U1.14 (VCC), U2.8 (V+), U4.11 (V+), U5.11 (V+), U6.11 (V+), C19.1, C20.1, C22.1, C24.1, C26.1, C28.1, C30.1, D7.1 (K), R63.1, RV7.1, U3.4 (V+)
- net -12V: now also R24.2, R58.2, U2.4 (V-), U4.6 (V-), U5.6 (V-), U6.6 (V-), C21.2, C23.2, C25.2, C27.2, C29.2, C31.2, D8.2 (A), R64.2, U3.11 (V-); no longer C1.1, C2.2, C3.1, Q1.2 (B), R7.2, R9.2
- net GND: now also C1.1, C2.2, C3.1, Q1.2 (B), R7.2, R9.2, U1.7 (GND), U2.5 (+), C12.2, C19.2, C20.2, C21.1, C22.2, C23.1, C24.2, C25.1, C26.2, C27.1, C28.2, C29.1, C30.2, C31.1, D10.2 (A), D6.1 (K), D9.1 (K), J4.S, J6.S, J7.3 (Pin_3), J7.4 (Pin_4), J7.5 (Pin_5), J7.6 (Pin_6), J7.7 (Pin_7), J7.8 (Pin_8), Q5.2 (B), Q6.2 (B), R60.2, RV10.1, RV12.1, RV5.3, RV7.3, RV9.2, RV9.3, U3.10 (+)
- net at R47.1, R51.1: now also R50.2, R55.1, U5.8, U6.4 (-), R59.1, TP10.1; no longer U6.13 (-)
- net at C8.2, RV6.1: now also TP4.1
- net at C2.1: now also SW1.1 (A)
- net at U5.5, U5.7: now also C17.2; no longer C16.2
- net at R49.2, R54.1, R57.1: now also U4.8; no longer U5.8
- net at R4.1: now also U1.10; no longer U1.3
- net at R4.2, RV2.2, RV2.3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: now also TP3.1
- net at U2.6 (-): now also C11.1, R13.2, R17.2, R18.2, R19.1, R33.1
- net at U2.7: now also C11.2, Q4.2 (B)
- net at U4.5, U4.7: now also C16.2
- net at R37.2: now also C15.1, D5.1 (K), U6.9, U3.5 (+); no longer U4.8
- net at R40.2, R45.1: now also U4.3 (+); no longer U5.3 (+)
- net at C3.2, R1.1, U1.5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: now also RV5.1, SW1.2 (B)
- net at R41.2, R46.1: now also U5.3 (+); no longer U6.3 (+)
- net at R26.1, R31.1, U4.13 (-): now also R61.1
- net at C9.2, R15.1: now also R44.1, U1.1, U1.2, TP5.1, U3.3 (+); no longer U1.8, U1.9
- net at D3.2 (A), J3.T: no longer J1.2 (Pin_2), J2.2 (Pin_2)
- net at U6.10, U6.12: no longer R52.1
- net at C1.2, R2.1: now also U1.8, U1.9; no longer U1.1, U1.2
- net at R16.2, U2.1: now also C10.1
- net at U6.5, U6.7: now also R51.2, R52.1; no longer C17.2
- net at R34.2, R37.1: now also U6.13 (-); no longer U4.4 (-)
- net I_FREQ: now reaches U4.1
- net I_FREQ: now also U4.16, U5.1, U5.16, R23.2
- net at R36.2: now also U6.14 (+); no longer U4.3 (+)
- net at R48.1: now also U6.3 (+); no longer U6.14 (+)
- net at U6.16: now also Q5.3 (C)
- net at U1.13: now also U1.3; no longer U1.10
- net at R20.1, RV8.2: now also R21.2
- net at C6.2, Q3.2 (B): now also C4.2, C5.2, TP1.1
- net at R42.1, R49.1: now also U4.4 (-); no longer U5.4 (-)
- net at R43.1, R50.1: now also U5.4 (-); no longer U6.4 (-)
- net at U6.1: now also Q6.3 (C)
- net at R28.1, U4.14 (+): now also C10.2, TP6.1
- net at R24.1: now also R21.1, R22.2, R30.1, U3.9 (-)
- net at R5.2, RV1.2, RV1.3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: now also TP2.1
- net at R62.2: now also J6.T
- new net: R30.2, R35.1, U3.8
- new net: R59.2, RV11.1
- new net: R61.2, RV11.2
- new net: R60.1, RV11.3
- new net: C18.1, R58.1, U6.8
- new net: C18.2, RV12.3, TP11.1
- new net: R53.1, R56.1, TP9.1, U3.6 (-), U3.7
- new net: D6.2 (A), R53.2
- new net: D10.1 (K), R64.1
- new net: C4.1, D1.1 (K)
- new net: D1.2 (A), J1.2 (Pin_2)
- new net: R18.1, RV7.2
- new net: R25.2, RV9.1
- new net: R33.2, RV10.2
- new net: J4.T, R17.1
- new net: D9.2 (A), R63.2
- new net: C12.1, D4.1 (K), R25.1, U3.12 (+)
- new net: D4.2 (A), U3.1, U3.2 (-)
- new net: R13.1, RV5.2
- new net: C5.1, D2.1 (K)
- new net: D2.2 (A), J2.2 (Pin_2)
- new net: Q6.1 (E), R56.2
- new net: Q4.3 (C), R23.1, TP7.1
- new net: RV10.3, TP8.1, U3.13 (-), U3.14
- new net: Q4.1 (E), R19.2
- new net: Q5.1 (E), R35.2
- new net: D7.2 (A), J7.1 (Pin_1), J7.2 (Pin_2)
- new net: D8.1 (K), J7.10 (Pin_10), J7.9 (Pin_9)
- new net: R62.1, RV12.2
- no-connect marks 8 -> 10
Other:
- note added: "Filter Env Amount"
- note added: "Filter Env Decay"
- note added: "Freq LFO Mod"
- note added: "Volume Env Decay"
- note removed: "Non Voltage Controlled Envelope"
- title: (none) -> Magnum Percussion Instrument
- moved on the sheet: C1, C13, C14, C15, C16, C17, C2, C3, C6, C7, C8, C9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
