File: filter.kicad_sch (KiCad schematic)
At the start: 31 parts, among them U5 LM13700, U6 LM13700

Commit message: Updating after tweaks and project improvements
Parts:
- C17, C18, C19, C20: value 150pF (poly) -> 100pF (poly); footprint Rumblesan_Footprints:C_Rect_L7.0mm_W3.5mm_P5.00mm -> rumblesan-standard-parts:C_Rect_L7.0mm_W3.5mm_P5.00mm
- R43, R44, R45, R46, R47, R48, R49, R50, R51, R54, R55, R56, R57, R58, R59, R60, R61, R62, R63, R66, R67: footprint Rumblesan_Footprints:Resistor_THT_L6.3mm_D2.5mm_P10.16mm_Horizontal -> rumblesan-standard-parts:R_Axial_DIN0207_L6.3mm_D2.5mm_P10.16mm_Horizontal
- R52, R53, R64, R65: value 21k -> 22k; footprint Rumblesan_Footprints:Resistor_THT_L6.3mm_D2.5mm_P10.16mm_Horizontal -> rumblesan-standard-parts:R_Axial_DIN0207_L6.3mm_D2.5mm_P10.16mm_Horizontal
- U5, U6: footprint Package_DIP:DIP-16_W7.62mm_LongPads -> rumblesan-standard-parts:DIP-16_W7.62mm_Socket
Other:
- title: (none) -> Magnum Percussion Instrument

Commit message: Further tweaks and layout improvements
Parts:
- C17, C18, C19, C20: value 100pF (poly) -> 100pF; Spec (none) -> film polypropylene; Tolerance (none) -> 5%
- R43, R44, R45, R46, R47, R48, R49, R50, R51, R52, R53, R54, R55, R56, R57, R58, R59, R60, R61, R62, R63, R64, R65, R66, R67: Tolerance (none) -> 1%
