File: magnum-drum-synth.kicad_sch (KiCad schematic)
At the start: 148 parts, among them J1 Input1, J2 Input1, J3 Trig_In, J4 Freq_CV, J5 Decay_CV, J6 Audio_Out, J7 Euro_Power, Q1 2N3904, Q2 2N3904, Q3 2N3904, Q4 2N3906, Q5 2N3906, Q6 2N3906, SW1 SW_SPDT, U1 HEF4093B, U2 TL072, U3 TL074, U4 LM13700, U5 LM13700, U6 LM13700

Commit message: Update schematic
Other:
- note added: "Filter Envelope"
- moved on the sheet: C1, C11, C12, C15, C18, C19, C2, C20, C21, C22, C23, C24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

Commit message: Creating rev02
Parts:
- removed C13, C17: 1nF, Rumblesan_Footprints:C_Rect_L7.0mm_W3.5mm_P2.50mm_P5.00mm, symbol Device:C
- removed C18: 10uF, Capacitor_THT:CP_Radial_D5.0mm_P2.50mm, symbol Device:C_Polarized
- removed C19, C22, C23, C24, C25, C26, C27, C28, C29, C30, C31: 100nF (X7R), Rumblesan_Footprints:C_Rect_L7.0mm_W3.5mm_P2.50mm_P5.00mm, symbol Device:C
- removed C20, C21: 1uF, Capacitor_THT:CP_Radial_D5.0mm_P2.50mm, symbol Device:C_Polarized
- removed C4, C5, C6: 100nF, Rumblesan_Footprints:C_Rect_L7.0mm_W3.5mm_P2.50mm_P5.00mm, symbol Device:C
- removed D10, D6, D9: LED, LED_THT:LED_D5.0mm, symbol Device:LED
- removed D2: D, Rumblesan_Footprints:Diode_THT_P7.62mm_Horizontal, symbol Device:D
- removed D7, D8: 1N5189, Rumblesan_Footprints:D_DO-35_SOD27_P7.62mm_Horizontal, symbol Device:D
- removed J2: Input1, Connector_PinHeader_2.54mm:PinHeader_1x02_P2.54mm_Vertical, symbol Connector:Conn_01x02_Female
- removed J7: Euro_Power, EurorackBasics:EurorackPowerHeader_2x05_P2.54mm_Shrouded, symbol Connector_Generic:Conn_02x05_Odd_Even
- removed Q4: 2N3906, Package_TO_SOT_THT:TO-92_Inline_Wide, symbol Transistor_BJT:2N3906
- removed R23, R31, R40, R49, R50, R51, R57: 100k, Resistor_THT:R_Axial_DIN0207_L6.3mm_D2.5mm_P7.62mm_Horizontal, symbol Device:R
- removed R26, R27, R42, R43, R45, R46, R47, R48: 220r, Resistor_THT:R_Axial_DIN0207_L6.3mm_D2.5mm_P7.62mm_Horizontal, symbol Device:R
- removed R38, R39, R52, R54, R55, R58, R59: 10k, Resistor_THT:R_Axial_DIN0207_L6.3mm_D2.5mm_P7.62mm_Horizontal, symbol Device:R
- removed R4, R5: 100r, Resistor_THT:R_Axial_DIN0207_L6.3mm_D2.5mm_P7.62mm_Horizontal, symbol Device:R
- removed R53: R, Resistor_THT:R_Axial_DIN0207_L6.3mm_D2.5mm_P7.62mm_Horizontal, symbol Device:R
- removed R60, R62: 1k, Resistor_THT:R_Axial_DIN0207_L6.3mm_D2.5mm_P7.62mm_Horizontal, symbol Device:R
- removed R61: 6k8, Resistor_THT:R_Axial_DIN0207_L6.3mm_D2.5mm_P7.62mm_Horizontal, symbol Device:R
- removed R63, R64: 3k3, Resistor_THT:R_Axial_DIN0207_L6.3mm_D2.5mm_P7.62mm_Horizontal, symbol Device:R
- removed RV11: 50kA, Rumblesan_Footprints:Potentiometer_Alpha_RD901F-40-00D_Single_Vertical_CircularHoles, symbol Device:R_Potentiometer
- removed SW1: SW_SPDT, Rumblesan_Footprints:SW_SPDT_DailyWell_MiniToggle, symbol Switch:SW_SPDT
- removed TP10, TP11: TestPoint, TestPoint:TestPoint_Loop_D2.50mm_Drill1.0mm_LowProfile, symbol Connector:TestPoint
- removed unit 5 of U1
- removed unit 3 of U2
- removed unit 1 of U2
- removed unit 5 of U3
- removed U4, U5, U6: LM13700, Package_DIP:DIP-16_W7.62mm_LongPads, symbol Amplifier_Operational:LM13700
- added C10: 22pF, Rumblesan_Footprints:C_Rect_L7.0mm_W3.5mm_P5.00mm, symbol Device:C
- added C6, C7: 1uF, Capacitor_THT:CP_Radial_D5.0mm_P2.50mm, symbol Device:C_Polarized
- added C8: 220nF, Rumblesan_Footprints:C_Rect_L7.0mm_W3.5mm_P5.00mm, symbol Device:C
- added D3, D4: 1n4148, Rumblesan_Footprints:Diode_THT_P7.62mm_Horizontal, symbol Device:D
- added H1, H2, H3, H4, H5, H6: MouseBite, Panelization:mouse-bite-2mm-slot, symbol Panelization:MouseBite
- added H10, H7, H8, H9: MountingHole_Pad, MountingHole:MountingHole_3.2mm_M3_ISO7380_Pad, symbol Mechanical:MountingHole_Pad
- added J10: Filter_Mod_Main, Connector_PinSocket_2.54mm:PinSocket_1x04_P2.54mm_Vertical, symbol Connector:Conn_01x04_Male
- added J11: Filter_Mod_Ctrl, Connector_PinSocket_2.54mm:PinSocket_1x04_P2.54mm_Vertical, symbol Connector:Conn_01x04_Female
- added J20: Amp_Decay_Ctrl, Connector_PinSocket_2.54mm:PinSocket_1x02_P2.54mm_Vertical, symbol Connector:Conn_01x02_Female
- added J21: Amp_Decay_Main, Connector_PinHeader_2.54mm:PinHeader_1x02_P2.54mm_Vertical, symbol Connector:Conn_01x02_Male
- added J22: Res_Main, Connector_PinHeader_2.54mm:PinHeader_1x02_P2.54mm_Vertical, symbol Connector:Conn_01x02_Female
- added J23: Res_Ctrl, Connector_PinSocket_2.54mm:PinSocket_1x02_P2.54mm_Vertical, symbol Connector:Conn_01x02_Male
- added J3: Trig_Ctrl, Connector_PinSocket_2.54mm:PinSocket_1x04_P2.54mm_Vertical, symbol Connector:Conn_01x04_Female
- added J4: Trig_Main, Connector_PinHeader_2.54mm:PinHeader_1x04_P2.54mm_Vertical, symbol Connector:Conn_01x04_Male
- added J5: Tap_Normal, Connector_PinHeader_2.54mm:PinHeader_1x03_P2.54mm_Vertical, symbol Connector:Conn_01x03_Male
- added J6, J7: Signals_Main, Connector_PinSocket_2.54mm:PinSocket_1x06_P2.54mm_Vertical, symbol Connector:Conn_01x06_Male
- added J8: Osc_Freq_Main, Connector_PinHeader_2.54mm:PinHeader_1x06_P2.54mm_Vertical, symbol Connector:Conn_01x06_Male
- added J9: Osc_Freq_Ctrl, Connector_PinSocket_2.54mm:PinSocket_1x06_P2.54mm_Vertical, symbol Connector:Conn_01x06_Female
- added Q3, Q5: 2N3904, Package_TO_SOT_THT:TO-92_Inline_Wide, symbol Transistor_BJT:2N3904
- added Q6: 2N3906, Package_TO_SOT_THT:TO-92_Inline_Wide, symbol Transistor_BJT:2N3906
- added R10, R6, R9: 10k, Rumblesan_Footprints:Resistor_THT_L6.3mm_D2.5mm_P10.16mm_Horizontal, symbol Device:R
- added R11: 1m, Rumblesan_Footprints:Resistor_THT_L6.3mm_D2.5mm_P10.16mm_Horizontal, symbol Device:R
- added R17: 100k, Rumblesan_Footprints:Resistor_THT_L6.3mm_D2.5mm_P10.16mm_Horizontal, symbol Device:R
- added R21: 150k, Rumblesan_Footprints:Resistor_THT_L6.3mm_D2.5mm_P10.16mm_Horizontal, symbol Device:R
- added R34: 20k, Rumblesan_Footprints:Resistor_THT_L6.3mm_D2.5mm_P10.16mm_Horizontal, symbol Device:R
- added R35: 2k, Rumblesan_Footprints:Resistor_THT_L6.3mm_D2.5mm_P10.16mm_Horizontal, symbol Device:R
- added RV1: 100k, Rumblesan_Footprints:Potentiometer_THT_Bourns_3306P_Vertical, symbol Device:R_Potentiometer_Trim
- added SW1: SW_DPDT_x2, Rumblesan_Footprints:SW_PUSH_2P2T_8mm_Apem_MHPS2285, symbol Switch:SW_DPDT_x2
- added U2: TL072, Package_DIP:DIP-8_W7.62mm_LongPads, symbol Amplifier_Operational:TL072
- added unit 1 of U3
- added U7: LM13700, Package_DIP:DIP-16_W7.62mm_LongPads, symbol Amplifier_Operational:LM13700
- C12: renamed from C11; value 47pF -> 10nF; footprint Rumblesan_Footprints:C_Rect_L7.0mm_W3.5mm_P2.50mm_P5.00mm -> Rumblesan_Footprints:C_Rect_L7.0mm_W3.5mm_P5.00mm
- C14: value 1nF -> 22pF; footprint Rumblesan_Footprints:C_Rect_L7.0mm_W3.5mm_P2.50mm_P5.00mm -> Rumblesan_Footprints:C_Rect_L7.0mm_W3.5mm_P5.00mm
- C15: value 1uF -> 10uF
- C16: value 1nF -> 1uF; footprint Rumblesan_Footprints:C_Rect_L7.0mm_W3.5mm_P2.50mm_P5.00mm -> Capacitor_THT:C_Radial_D6.3mm_H7.0mm_P2.50mm
- C2: renamed from C1; footprint Rumblesan_Footprints:C_Rect_L7.0mm_W3.5mm_P2.50mm_P5.00mm -> Rumblesan_Footprints:C_Rect_L7.0mm_W3.5mm_P5.00mm
- C3: footprint Rumblesan_Footprints:C_Rect_L7.0mm_W3.5mm_P2.50mm_P5.00mm -> Rumblesan_Footprints:C_Rect_L7.0mm_W3.5mm_P5.00mm
- C4: renamed from C7; footprint Rumblesan_Footprints:C_Rect_L7.0mm_W3.5mm_P2.50mm_P5.00mm -> Rumblesan_Footprints:C_Rect_L7.0mm_W3.5mm_P5.00mm
- C5: renamed from C8; footprint Rumblesan_Footprints:C_Rect_L7.0mm_W3.5mm_P2.50mm_P5.00mm -> Rumblesan_Footprints:C_Rect_L7.0mm_W3.5mm_P5.00mm
- C9: value 100nF -> 220nF; footprint Rumblesan_Footprints:C_Rect_L7.0mm_W3.5mm_P2.50mm_P5.00mm -> Rumblesan_Footprints:C_Rect_L7.0mm_W3.5mm_P5.00mm
- D1: value D -> 1n4148
- D2: renamed from D3; value D -> 1n4148
- D5: renamed from D4; value D -> 1n4148
- D6: renamed from D5; value D -> 1n4148
- J1: value Input1 -> Piezo
- J12: renamed from J4; footprint AudioJacks:Jack_3.5mm_QingPu_WQP-PJ398SM_Vertical -> EurorackBasics:Jack_3.5mm_QingPu_WQP-PJ398SM_Vertical
- J18: renamed from J5; footprint AudioJacks:Jack_3.5mm_QingPu_WQP-PJ398SM_Vertical -> EurorackBasics:Jack_3.5mm_QingPu_WQP-PJ398SM_Vertical
- J2: renamed from J3; footprint AudioJacks:Jack_3.5mm_QingPu_WQP-PJ398SM_Vertical -> EurorackBasics:Jack_3.5mm_QingPu_WQP-PJ398SM_Vertical
- J26: renamed from J6; footprint AudioJacks:Jack_3.5mm_QingPu_WQP-PJ398SM_Vertical -> EurorackBasics:Jack_3.5mm_QingPu_WQP-PJ398SM_Vertical
- R1: renamed from R3; footprint Resistor_THT:R_Axial_DIN0207_L6.3mm_D2.5mm_P7.62mm_Horizontal -> Rumblesan_Footprints:Resistor_THT_L6.3mm_D2.5mm_P10.16mm_Horizontal
- R12: value 100k -> 220k; footprint Resistor_THT:R_Axial_DIN0207_L6.3mm_D2.5mm_P7.62mm_Horizontal -> Rumblesan_Footprints:Resistor_THT_L6.3mm_D2.5mm_P10.16mm_Horizontal
- R13: renamed from R10; value R -> 10k; footprint Resistor_THT:R_Axial_DIN0207_L6.3mm_D2.5mm_P7.62mm_Horizontal -> Rumblesan_Footprints:Resistor_THT_L6.3mm_D2.5mm_P10.16mm_Horizontal
- R14: renamed from R15; value R -> 100k; footprint Resistor_THT:R_Axial_DIN0207_L6.3mm_D2.5mm_P7.62mm_Horizontal -> Rumblesan_Footprints:Resistor_THT_L6.3mm_D2.5mm_P10.16mm_Horizontal
- R15: renamed from R14; footprint Resistor_THT:R_Axial_DIN0207_L6.3mm_D2.5mm_P7.62mm_Horizontal -> Rumblesan_Footprints:Resistor_THT_L6.3mm_D2.5mm_P10.16mm_Horizontal
- R16: renamed from R11; footprint Resistor_THT:R_Axial_DIN0207_L6.3mm_D2.5mm_P7.62mm_Horizontal -> Rumblesan_Footprints:Resistor_THT_L6.3mm_D2.5mm_P10.16mm_Horizontal
- R18: renamed from R16; footprint Resistor_THT:R_Axial_DIN0207_L6.3mm_D2.5mm_P7.62mm_Horizontal -> Rumblesan_Footprints:Resistor_THT_L6.3mm_D2.5mm_P10.16mm_Horizontal
- R19: renamed from R18; footprint Resistor_THT:R_Axial_DIN0207_L6.3mm_D2.5mm_P7.62mm_Horizontal -> Rumblesan_Footprints:Resistor_THT_L6.3mm_D2.5mm_P10.16mm_Horizontal
- R2, R32: footprint Resistor_THT:R_Axial_DIN0207_L6.3mm_D2.5mm_P7.62mm_Horizontal -> Rumblesan_Footprints:Resistor_THT_L6.3mm_D2.5mm_P10.16mm_Horizontal
- R20: renamed from R17; footprint Resistor_THT:R_Axial_DIN0207_L6.3mm_D2.5mm_P7.62mm_Horizontal -> Rumblesan_Footprints:Resistor_THT_L6.3mm_D2.5mm_P10.16mm_Horizontal
- R22: renamed from R33; footprint Resistor_THT:R_Axial_DIN0207_L6.3mm_D2.5mm_P7.62mm_Horizontal -> Rumblesan_Footprints:Resistor_THT_L6.3mm_D2.5mm_P10.16mm_Horizontal
- R23: renamed from R13; footprint Resistor_THT:R_Axial_DIN0207_L6.3mm_D2.5mm_P7.62mm_Horizontal -> Rumblesan_Footprints:Resistor_THT_L6.3mm_D2.5mm_P10.16mm_Horizontal
- R24: renamed from R19; value 100k -> 2k; footprint Resistor_THT:R_Axial_DIN0207_L6.3mm_D2.5mm_P7.62mm_Horizontal -> Rumblesan_Footprints:Resistor_THT_L6.3mm_D2.5mm_P10.16mm_Horizontal
- R25: renamed from R20; footprint Resistor_THT:R_Axial_DIN0207_L6.3mm_D2.5mm_P7.62mm_Horizontal -> Rumblesan_Footprints:Resistor_THT_L6.3mm_D2.5mm_P10.16mm_Horizontal
- R26: renamed from R25; value R -> 1k; footprint Resistor_THT:R_Axial_DIN0207_L6.3mm_D2.5mm_P7.62mm_Horizontal -> Rumblesan_Footprints:Resistor_THT_L6.3mm_D2.5mm_P10.16mm_Horizontal
- R27: renamed from R21; footprint Resistor_THT:R_Axial_DIN0207_L6.3mm_D2.5mm_P7.62mm_Horizontal -> Rumblesan_Footprints:Resistor_THT_L6.3mm_D2.5mm_P10.16mm_Horizontal
- R28: value 220r -> 51r; footprint Resistor_THT:R_Axial_DIN0207_L6.3mm_D2.5mm_P7.62mm_Horizontal -> Rumblesan_Footprints:Resistor_THT_L6.3mm_D2.5mm_P10.16mm_Horizontal
- R29: value 220r -> 470r; footprint Resistor_THT:R_Axial_DIN0207_L6.3mm_D2.5mm_P7.62mm_Horizontal -> Rumblesan_Footprints:Resistor_THT_L6.3mm_D2.5mm_P10.16mm_Horizontal
- R3: renamed from R1; footprint Resistor_THT:R_Axial_DIN0207_L6.3mm_D2.5mm_P7.62mm_Horizontal -> Rumblesan_Footprints:Resistor_THT_L6.3mm_D2.5mm_P10.16mm_Horizontal
- R30: renamed from R22; footprint Resistor_THT:R_Axial_DIN0207_L6.3mm_D2.5mm_P7.62mm_Horizontal -> Rumblesan_Footprints:Resistor_THT_L6.3mm_D2.5mm_P10.16mm_Horizontal
- R31: renamed from R24; footprint Resistor_THT:R_Axial_DIN0207_L6.3mm_D2.5mm_P7.62mm_Horizontal -> Rumblesan_Footprints:Resistor_THT_L6.3mm_D2.5mm_P10.16mm_Horizontal
- R33: renamed from R30; footprint Resistor_THT:R_Axial_DIN0207_L6.3mm_D2.5mm_P7.62mm_Horizontal -> Rumblesan_Footprints:Resistor_THT_L6.3mm_D2.5mm_P10.16mm_Horizontal
- R36: renamed from R34; footprint Resistor_THT:R_Axial_DIN0207_L6.3mm_D2.5mm_P7.62mm_Horizontal -> Rumblesan_Footprints:Resistor_THT_L6.3mm_D2.5mm_P10.16mm_Horizontal
- R37: renamed from R35; footprint Resistor_THT:R_Axial_DIN0207_L6.3mm_D2.5mm_P7.62mm_Horizontal -> Rumblesan_Footprints:Resistor_THT_L6.3mm_D2.5mm_P10.16mm_Horizontal
- R38: renamed from R44; value R -> 680r; footprint Resistor_THT:R_Axial_DIN0207_L6.3mm_D2.5mm_P7.62mm_Horizontal -> Rumblesan_Footprints:Resistor_THT_L6.3mm_D2.5mm_P10.16mm_Horizontal
- R39: renamed from R36; footprint Resistor_THT:R_Axial_DIN0207_L6.3mm_D2.5mm_P7.62mm_Horizontal -> Rumblesan_Footprints:Resistor_THT_L6.3mm_D2.5mm_P10.16mm_Horizontal
- R4: renamed from R6; footprint Resistor_THT:R_Axial_DIN0207_L6.3mm_D2.5mm_P7.62mm_Horizontal -> Rumblesan_Footprints:Resistor_THT_L6.3mm_D2.5mm_P10.16mm_Horizontal
- R40: renamed from R37; footprint Resistor_THT:R_Axial_DIN0207_L6.3mm_D2.5mm_P7.62mm_Horizontal -> Rumblesan_Footprints:Resistor_THT_L6.3mm_D2.5mm_P10.16mm_Horizontal
- R41: value 100k -> 1k; footprint Resistor_THT:R_Axial_DIN0207_L6.3mm_D2.5mm_P7.62mm_Horizontal -> Rumblesan_Footprints:Resistor_THT_L6.3mm_D2.5mm_P10.16mm_Horizontal
- R42: renamed from R56; value R -> 33k; footprint Resistor_THT:R_Axial_DIN0207_L6.3mm_D2.5mm_P7.62mm_Horizontal -> Rumblesan_Footprints:Resistor_THT_L6.3mm_D2.5mm_P10.16mm_Horizontal
- R5: renamed from R7; footprint Resistor_THT:R_Axial_DIN0207_L6.3mm_D2.5mm_P7.62mm_Horizontal -> Rumblesan_Footprints:Resistor_THT_L6.3mm_D2.5mm_P10.16mm_Horizontal
- R7: renamed from R8; footprint Resistor_THT:R_Axial_DIN0207_L6.3mm_D2.5mm_P7.62mm_Horizontal -> Rumblesan_Footprints:Resistor_THT_L6.3mm_D2.5mm_P10.16mm_Horizontal
- R8: renamed from R9; footprint Resistor_THT:R_Axial_DIN0207_L6.3mm_D2.5mm_P7.62mm_Horizontal -> Rumblesan_Footprints:Resistor_THT_L6.3mm_D2.5mm_P10.16mm_Horizontal
- RV2: renamed from RV4; footprint Rumblesan_Footprints:Potentiometer_Alpha_RD901F-40-00D_Single_Vertical_CircularHoles -> Rumblesan_Footprints:Potentiometer_Alpha_RD901F-40-00D_Single_Vertical; Name (none) -> OSC2 Level
- RV3: renamed from RV2; footprint Rumblesan_Footprints:Potentiometer_Alpha_RD901F-40-00D_Single_Vertical_CircularHoles -> Rumblesan_Footprints:Potentiometer_Alpha_RD901F-40-00D_Single_Vertical
- RV4: renamed from RV1; footprint Rumblesan_Footprints:Potentiometer_Alpha_RD901F-40-00D_Single_Vertical_CircularHoles -> Rumblesan_Footprints:Potentiometer_Alpha_RD901F-40-00D_Single_Vertical
- RV5: renamed from RV3; footprint Rumblesan_Footprints:Potentiometer_Alpha_RD901F-40-00D_Single_Vertical_CircularHoles -> Rumblesan_Footprints:Potentiometer_Alpha_RD901F-40-00D_Single_Vertical; Name (none) -> OSC1 Level
- RV6: footprint Rumblesan_Footprints:Potentiometer_Alpha_RD901F-40-00D_Single_Vertical_CircularHoles -> Rumblesan_Footprints:Potentiometer_Alpha_RD901F-40-00D_Single_Vertical; Name (none) -> Noise Level
- TP1: renamed from TP4; value TestPoint -> Noise TestPoint
- TP2: renamed from TP3; value TestPoint -> OSC1 TestPoint
- TP3: renamed from TP2; value TestPoint -> OSC2 TestPoint
- TP4: renamed from TP1; value TestPoint -> Trigger TestPoint
- TP5: value TestPoint -> Schmitt Trigger TestPoint
- TP6: value TestPoint -> Mixer TestPoint
- TP8: value TestPoint -> Filter Env TestPoint
- renumbered C2 to C1, C10 to C11, C12 to C13, Q3 to Q4, Q5 to Q7, Q6 to Q8, RV8 to RV10, RV9 to RV11, RV10 to RV7, RV7 to RV8, RV5 to RV9, U2 to U3, U3 to U4
Connections:
- net +12V: now also D1.1 (K), RV8.3, Q3.3 (C), Q5.3 (C); no longer RV8.1
- net -12V: now also R31.1, R32.1, R21.1, R9.2; no longer R31.2
- net GND: now also C16.2, C3.2, D2.2 (A), RV2.1, RV5.1, RV6.1, RV8.1, RV9.1, U4.3 (+), C8.1, H10.1, H7.1, H8.1, H9.1, Q6.1 (E), R10.1, R11.2, R35.2, RV1.1, U2.5 (+); no longer C14.1, C15.2, C16.1, C3.1, R28.2, RV12.1, RV2.3, RV5.3, RV6.3, RV8.3, RV9.3, U4.10 (+)
- net at R27.1, R30.2, R33.1: now also C14.1, R31.2, U4.2 (-); no longer R31.1, U4.9 (-)
- net at R33.2, R37.1: now also C14.2, U4.1; no longer U4.8
- net OSC2_LFO_Cap: now reaches C1.1
- net OSC2_LFO_Cap: now also J8.1 (Pin_1)
- net Noise_Signal: now reaches C5.2, TP1.1
- net Noise_Signal: now also J6.3 (Pin_3); no longer RV6.1
- net at RV12.3: now also J23.1 (Pin_1)
- net at C11.1, R18.2: now also C10.2, U2.7
- net Filter/Input: now reaches C11.2, TP6.1
- net Filter/Input: no longer R28.1
- net at Q4.2 (B), TP4.1: now also D3.1 (K), D4.1 (K)
- net OSC1_Freq_R: now reaches U1.10
- net OSC1_Freq_R: now also C6.1, J8.5 (Pin_5)
- net at D1.2 (A), J1.2 (Pin_2): now also D2.1 (K), R6.1
- net at C12.1, R19.2, R20.2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: now also R22.2, R21.2; no longer R22.1
- net Freq_Control_Ctrl: now reaches C12.2, U3.7
- net Freq_Control_Ctrl: now also R24.2, J11.3 (Pin_3)
- net Final_Output_Main: now reaches R41.2
- net Final_Output_Main: now also J4.4 (Pin_4)
- net Filter_Env_Decay: now reaches R26.2
- net Filter_Env_Decay: now also J10.2 (Pin_2); no longer RV11.1
- net at RV7.2: now also R23.1; no longer R22.2
- net at RV5.2: now also J7.6 (Pin_6); no longer R16.1
- net at R15.2, R16.2, R18.1: now also C10.1, R17.2, U2.6 (-); no longer R12.2
- net Trigger: now reaches C9.2, R14.1, R38.1, TP5.1, U1.1, U1.2
- net Trigger: now also U4.12 (+); no longer U4.3 (+)
- net at RV6.2: now also J7.4 (Pin_4); no longer R15.1
- net at D6.1 (K), U4.5 (+): now also C16.1, U7.5, U7.7; no longer C15.1, R40.2
- net at R32.2: now also Q5.1 (E), Q6.2 (B); no longer R41.1
- net at C13.1, D5.1 (K), R26.1: now also U4.10 (+); no longer U4.12 (+)
- net at U1.3: now also U1.5; no longer U1.13
- net at Q4.3 (C), R13.2: now also U1.6; no longer U1.12
- net at RV9.2: now also R22.1; no longer R23.1
- net at C9.1: now also U1.4; no longer U1.11
- net at R36.2, R40.1: now also U7.4 (-)
- net at R39.2: now also U7.3 (+)
- net at Q7.3 (C): now also U7.1
- net Final_Output_Ctrl: now reaches J26.T
- net Final_Output_Ctrl: now also J3.4 (Pin_4)
- net Freq_Control_Main: now reaches TP7.1
- net Freq_Control_Main: now also R28.1, J10.3 (Pin_3)
- net at R25.1, RV10.2: now also J20.2 (Pin_2); no longer R27.2
- net at U4.13 (-), U4.14: now also D5.2 (A); no longer RV7.3, TP8.1
- net at R30.1: now also J21.1 (Pin_1); no longer J18.T
- net OutputVCA/I_Gain: now reaches Q8.3 (C)
- net at R29.1: now also R28.2, Q5.2 (B)
- net at J2.T: now also J3.3 (Pin_3); no longer D2.2 (A)
- net at R12.1: now also J3.1 (Pin_1), U3.1; no longer RV2.2
- net at RV12.2: now also J23.2 (Pin_2)
- net at J2.TN: now also J3.2 (Pin_2)
- net at RV3.1: now also RV3.2, J9.5 (Pin_5); no longer R2.2
- net at RV4.1: now also RV4.2, J9.3 (Pin_3); no longer R3.2
- new net: J9.1 (Pin_1), SW1.1 (A)
- new net: J9.2 (Pin_2), SW1.2 (B)
- new net: J9.4 (Pin_4), RV4.3
- new net: J9.6 (Pin_6), RV3.3
- new net: D3.2 (A), J5.1 (Pin_1)
- new net: R35.1, RV12.1
- new net: C8.2, R11.1, RV1.2, U3.3 (+)
- new net: R40.2, U7.8
- new net: J7.3 (Pin_3), RV6.3
- new net: J11.4 (Pin_4), RV9.3
- new net: J7.2 (Pin_2), RV5.3
- new net: R10.2, R12.2, U3.2 (-)
- new net: D4.2 (A), J4.3 (Pin_3)
- new net: J21.2 (Pin_2), R27.2
- new net: J18.T, J20.1 (Pin_1)
- new net: J4.1 (Pin_1), J5.2 (Pin_2)
- new net: J4.2 (Pin_2), J5.3 (Pin_3)
- new net: R6.2, RV1.3
- new net: J7.5 (Pin_5), RV2.2
- new net: J7.1 (Pin_1), RV2.3
- new net Filter/I_Freq: Q6.3 (C)
- new net Filter/Output: C15.1, R34.1
- new net Filter_Env: J10.1 (Pin_1), TP8.1, U4.8, U4.9 (-)
- new net Filter_Env_Decay_Ctrl: J11.2 (Pin_2), RV11.1
- new net Filter_Env_Mod_Ctrl: J11.1 (Pin_1), RV7.3
- new net Noise_Return: J6.4 (Pin_4), R15.1
- new net OSC1_Freq_L: J8.6 (Pin_6), R2.2
- new net OSC1_Return: J6.6 (Pin_6), R16.1
- new net OSC1_Signal: C6.2, J6.2 (Pin_2), TP2.1
- new net OSC2_Freq_L: J8.3 (Pin_3), R3.2
- new net OSC2_Freq_R: C7.1, J8.4 (Pin_4), U1.11
- new net OSC2_LFO_Main: C3.1, J8.2 (Pin_2), Q3.2 (B), R3.1, U1.12, U1.13
- new net OSC2_LFO_Signal: J10.4 (Pin_4), Q3.1 (E), R9.1
- new net OSC2_Return: J6.5 (Pin_5), R17.1
- new net OSC2_Signal: C7.2, J6.1 (Pin_1), TP3.1
- new net OutputVCA/Input: C15.2
- new net OutputVCA/Output: R41.1
- new net Res_Amount: J22.2 (Pin_2)
- new net Res_Top: J22.1 (Pin_1), R34.2
- no-connect marks 10 -> 9
Other:
- added sheet Filter (filter.kicad_sch)
- added sheet OutputVCA (output-vca.kicad_sch)
- added sheet Power (power.kicad_sch)
- note added: "Select if connection to Trig in disables piezo"
- note removed: "Filter"
- note removed: "Filter Env Amount"
- note removed: "Filter Env Decay"
- note removed: "Freq LFO Mod"
- note removed: "LFO/OSC select"
- note removed: "Mixer"
- note removed: "Noise Level"
- note removed: "OSC1 Level"
- note removed: "OSC2 Level"
- note removed: "Output VCA"
- note removed: "Power connections"
- note removed: "Volume Env Decay"
- moved on the sheet: C1, C11, C12, C13, C2, C3, C4, C5, C9, D2, D5, D6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

Commit message: Updating after tweaks and project improvements
Parts:
- removed C11: 10uF, Capacitor_THT:CP_Radial_D5.0mm_P2.50mm, symbol Device:C_Polarized
- removed C9: 220nF, Rumblesan_Footprints:C_Rect_L7.0mm_W3.5mm_P5.00mm, symbol Device:C
- removed H1, H2, H3, H4, H5, H6: MouseBite, Panelization:mouse-bite-2mm-slot, symbol Panelization:MouseBite
- added C36: 22pF, rumblesan-standard-parts:C_Rect_L7.0mm_W3.5mm_P5.00mm, symbol Device:C
- added C9: 1uF, rumblesan-standard-parts:CP_Radial_D5.0mm_P2.00mm, symbol Device:C_Polarized
- added H1, H2, H3, H4: MountingScrew_M3, MountingHole:MountingHole_3.2mm_M3, symbol Board_Hardware:MountingScrew_M3
- added H5, H6: Standoff_F-F, symbol Board_Hardware:Standoff_F-F
- added Q9: 2N3906, rumblesan-standard-parts:TO-92_Inline_Wide, symbol Transistor_BJT:2N3906
- added R73: 22k, rumblesan-standard-parts:R_Axial_DIN0207_L6.3mm_D2.5mm_P10.16mm_Horizontal, symbol Device:R
- added R74: 82k, rumblesan-standard-parts:R_Axial_DIN0207_L6.3mm_D2.5mm_P10.16mm_Horizontal, symbol Device:R
- added TP10, TP11: Mixer TestPoint, rumblesan-standard-parts:TestPoint_Loop_D2.50mm_Drill1.0mm_LowProfile, symbol Connector:TestPoint
- added TP12: Schmitt Trigger TestPoint, rumblesan-standard-parts:TestPoint_Loop_D2.50mm_Drill1.0mm_LowProfile, symbol Connector:TestPoint
- C1, C13, C15, C6, C7: footprint Capacitor_THT:CP_Radial_D5.0mm_P2.50mm -> rumblesan-standard-parts:CP_Radial_D5.0mm_P2.00mm
- C10, C12, C14, C2, C3, C4, C8: footprint Rumblesan_Footprints:C_Rect_L7.0mm_W3.5mm_P5.00mm -> rumblesan-standard-parts:C_Rect_L7.0mm_W3.5mm_P5.00mm
- C16: value 1uF -> 1uF (non polarised); footprint Capacitor_THT:C_Radial_D6.3mm_H7.0mm_P2.50mm -> rumblesan-standard-parts:C_Radial_D5.0mm_H5.0mm_P2.00mm
- C5: value 100nF -> 100nF (X7R); footprint Rumblesan_Footprints:C_Rect_L7.0mm_W3.5mm_P5.00mm -> rumblesan-standard-parts:C_Rect_L7.0mm_W3.5mm_P5.00mm
- D1, D2, D3, D4, D5, D6: value 1n4148 -> 1N4148; footprint Rumblesan_Footprints:Diode_THT_P7.62mm_Horizontal -> rumblesan-standard-parts:D_DO-35_SOD27_P7.62mm_Horizontal
- H10, H7, H8, H9: footprint MountingHole:MountingHole_3.2mm_M3_ISO7380_Pad -> rumblesan-standard-parts:MountingHole_3.2mm_M3_DIN965_Pad; now left out of the parts list
- J1: now left out of the parts list
- J10: value Filter_Mod_Main -> Conn_01x04_Male; footprint Connector_PinSocket_2.54mm:PinSocket_1x04_P2.54mm_Vertical -> Connector_PinHeader_2.54mm:PinHeader_1x04_P2.54mm_Vertical; Name (none) -> Filter Mod Header Main
- J11: value Filter_Mod_Ctrl -> Conn_01x04_Female; Name (none) -> Filter Mod Header Ctrl
- J12: value Freq_CV -> AudioJack2_SwitchT; footprint EurorackBasics:Jack_3.5mm_QingPu_WQP-PJ398SM_Vertical -> rumblesan-standard-parts:Jack_3.5mm_QingPu_WQP-PJ398SM_Vertical; Name (none) -> Freq CV
- J18: value Decay_CV -> AudioJack2_SwitchT; footprint EurorackBasics:Jack_3.5mm_QingPu_WQP-PJ398SM_Vertical -> rumblesan-standard-parts:Jack_3.5mm_QingPu_WQP-PJ398SM_Vertical; Name (none) -> Decay CV
- J2: value Trig_In -> AudioJack2_SwitchT; footprint EurorackBasics:Jack_3.5mm_QingPu_WQP-PJ398SM_Vertical -> rumblesan-standard-parts:Jack_3.5mm_QingPu_WQP-PJ398SM_Vertical; Name (none) -> Trig In
- J20: value Amp_Decay_Ctrl -> Conn_01x02_Female; Name (none) -> Amp Decay Header Ctrl
- J21: value Amp_Decay_Main -> Conn_01x02_Male; Name (none) -> Amp Decay Header Main
- J22: value Res_Main -> Conn_01x02_Male; symbol Connector:Conn_01x02_Female -> Connector:Conn_01x02_Male; Name (none) -> Res Header Main
- J23: value Res_Ctrl -> Conn_01x02_Female; symbol Connector:Conn_01x02_Male -> Connector:Conn_01x02_Female; Name (none) -> Res Header Ctrl
- J26: value Audio_Out -> AudioJack2_SwitchT; footprint EurorackBasics:Jack_3.5mm_QingPu_WQP-PJ398SM_Vertical -> rumblesan-standard-parts:Jack_3.5mm_QingPu_WQP-PJ398SM_Vertical; Name (none) -> Audio Out
- J3: value Trig_Ctrl -> Conn_01x04_Female; Name (none) -> Trig Header Ctrl
- J4: value Trig_Main -> Conn_01x04_Male; Name (none) -> Trig Header Main
- J5: value Tap_Normal -> Conn_01x03_Male; Name (none) -> Piezo Normal
- J6: value Signals_Main -> Conn_01x06_Male; footprint Connector_PinSocket_2.54mm:PinSocket_1x06_P2.54mm_Vertical -> Connector_PinHeader_2.54mm:PinHeader_1x06_P2.54mm_Vertical; Name (none) -> Signals Header Main
- J7: value Signals_Main -> Conn_01x06_Female; symbol Connector:Conn_01x06_Male -> Connector:Conn_01x06_Female; Name (none) -> Signals Header Ctrl
- J8: value Osc_Freq_Main -> Conn_01x06_Male; Name (none) -> OSC Freq Header Main
- J9: value Osc_Freq_Ctrl -> Conn_01x06_Female; Name (none) -> OSC Freq Header Ctrl
- Q1, Q2, Q3, Q4, Q5, Q6, Q7, Q8: footprint Package_TO_SOT_THT:TO-92_Inline_Wide -> rumblesan-standard-parts:TO-92_Inline_Wide
- R1, R10, R11, R12, R13, R16, R17, R18, R19, R2, R20, R22, R24, R26, R27, R28, R29, R3, R30, R31, R32, R33, R36, R37, R39, R4, R40, R41, R42, R5, R8, R9: footprint Rumblesan_Footprints:Resistor_THT_L6.3mm_D2.5mm_P10.16mm_Horizontal -> rumblesan-standard-parts:R_Axial_DIN0207_L6.3mm_D2.5mm_P10.16mm_Horizontal
- R14: value 100k -> 150k; footprint Rumblesan_Footprints:Resistor_THT_L6.3mm_D2.5mm_P10.16mm_Horizontal -> rumblesan-standard-parts:R_Axial_DIN0207_L6.3mm_D2.5mm_P10.16mm_Horizontal
- R15: value 100k -> 22k; footprint Rumblesan_Footprints:Resistor_THT_L6.3mm_D2.5mm_P10.16mm_Horizontal -> rumblesan-standard-parts:R_Axial_DIN0207_L6.3mm_D2.5mm_P10.16mm_Horizontal
- R21: value 150k -> 220k; footprint Rumblesan_Footprints:Resistor_THT_L6.3mm_D2.5mm_P10.16mm_Horizontal -> rumblesan-standard-parts:R_Axial_DIN0207_L6.3mm_D2.5mm_P10.16mm_Horizontal
- R23: value 100k -> 82k; footprint Rumblesan_Footprints:Resistor_THT_L6.3mm_D2.5mm_P10.16mm_Horizontal -> rumblesan-standard-parts:R_Axial_DIN0207_L6.3mm_D2.5mm_P10.16mm_Horizontal
- R25: value 15k -> 22k; footprint Rumblesan_Footprints:Resistor_THT_L6.3mm_D2.5mm_P10.16mm_Horizontal -> rumblesan-standard-parts:R_Axial_DIN0207_L6.3mm_D2.5mm_P10.16mm_Horizontal
- R34: value 20k -> 10k; footprint Rumblesan_Footprints:Resistor_THT_L6.3mm_D2.5mm_P10.16mm_Horizontal -> rumblesan-standard-parts:R_Axial_DIN0207_L6.3mm_D2.5mm_P10.16mm_Horizontal
- R35: value 2k -> 47k; footprint Rumblesan_Footprints:Resistor_THT_L6.3mm_D2.5mm_P10.16mm_Horizontal -> rumblesan-standard-parts:R_Axial_DIN0207_L6.3mm_D2.5mm_P10.16mm_Horizontal
- R38: value 680r -> 470r; footprint Rumblesan_Footprints:Resistor_THT_L6.3mm_D2.5mm_P10.16mm_Horizontal -> rumblesan-standard-parts:R_Axial_DIN0207_L6.3mm_D2.5mm_P10.16mm_Horizontal
- R6: value 10k -> 1k; footprint Rumblesan_Footprints:Resistor_THT_L6.3mm_D2.5mm_P10.16mm_Horizontal -> rumblesan-standard-parts:R_Axial_DIN0207_L6.3mm_D2.5mm_P10.16mm_Horizontal
- R7: value 6k8 -> 10k; footprint Rumblesan_Footprints:Resistor_THT_L6.3mm_D2.5mm_P10.16mm_Horizontal -> rumblesan-standard-parts:R_Axial_DIN0207_L6.3mm_D2.5mm_P10.16mm_Horizontal
- RV1: footprint Rumblesan_Footprints:Potentiometer_THT_Bourns_3306P_Vertical -> rumblesan-standard-parts:Potentiometer_THT_Bourns_3306P_Vertical; Name (none) -> Piezo Sensitivity
- RV10: footprint Rumblesan_Footprints:Potentiometer_Alpha_RD901F-40-00D_Single_Vertical_CircularHoles -> rumblesan-standard-parts:Potentiometer_Alpha_RD901F-40-00D_Single_Vertical; Name (none) -> Amp Env Decay
- RV11: footprint Rumblesan_Footprints:Potentiometer_Alpha_RD901F-40-00D_Single_Vertical_CircularHoles -> rumblesan-standard-parts:Potentiometer_Alpha_RD901F-40-00D_Single_Vertical; Name (none) -> Filter Env Decay
- RV12: value 100kA -> 50kB; footprint Rumblesan_Footprints:Potentiometer_Alpha_RD901F-40-00D_Single_Vertical_CircularHoles -> rumblesan-standard-parts:Potentiometer_Alpha_RD901F-40-00D_Single_Vertical; Name (none) -> Filter Res
- RV2, RV5, RV6: footprint Rumblesan_Footprints:Potentiometer_Alpha_RD901F-40-00D_Single_Vertical -> rumblesan-standard-parts:Potentiometer_Song_Huei_R0904N_Single_Vertical
- RV3: footprint Rumblesan_Footprints:Potentiometer_Alpha_RD901F-40-00D_Single_Vertical -> rumblesan-standard-parts:Potentiometer_Song_Huei_R0904N_Single_Vertical; Name (none) -> OSC1 Freq
- RV4: footprint Rumblesan_Footprints:Potentiometer_Alpha_RD901F-40-00D_Single_Vertical -> rumblesan-standard-parts:Potentiometer_Song_Huei_R0904N_Single_Vertical; Name (none) -> OSC2 Freq
- RV7: footprint Rumblesan_Footprints:Potentiometer_Alpha_RD901F-40-00D_Single_Vertical_CircularHoles -> rumblesan-standard-parts:Potentiometer_Alpha_RD901F-40-00D_Single_Vertical; Name (none) -> Filter Env Mod
- RV8: footprint Rumblesan_Footprints:Potentiometer_Alpha_RD901F-40-00D_Single_Vertical_CircularHoles -> rumblesan-standard-parts:Potentiometer_Alpha_RD901F-40-00D_Single_Vertical; Name (none) -> Filter Freq
- RV9: footprint Rumblesan_Footprints:Potentiometer_Alpha_RD901F-40-00D_Single_Vertical_CircularHoles -> rumblesan-standard-parts:Potentiometer_Alpha_RD901F-40-00D_Single_Vertical; Name (none) -> Filter LFO Mod
- SW1: footprint Rumblesan_Footprints:SW_PUSH_2P2T_8mm_Apem_MHPS2285 -> rumblesan-standard-parts:SW_PUSH_2P2T_8mm_Apem_MHPS2285
- SW1: footprint Rumblesan_Footprints:SW_PUSH_2P2T_8mm_Apem_MHPS2285 -> rumblesan-standard-parts:SW_PUSH_2P2T_8mm_Apem_MHPS2285; Name (none) -> OSC2 LFO
- TP1, TP2, TP3, TP4, TP5, TP6, TP7, TP8, TP9: footprint TestPoint:TestPoint_Loop_D2.50mm_Drill1.0mm_LowProfile -> rumblesan-standard-parts:TestPoint_Loop_D2.50mm_Drill1.0mm_LowProfile; now left out of the parts list
- U1: value HEF4093B -> CD4093B; footprint Package_DIP:DIP-14_W7.62mm_LongPads -> rumblesan-standard-parts:DIP-14_W7.62mm_Socket
- U2, U3: footprint Package_DIP:DIP-8_W7.62mm_LongPads -> rumblesan-standard-parts:DIP-8_W7.62mm_Socket
- U4: footprint Package_DIP:DIP-14_W7.62mm_LongPads -> rumblesan-standard-parts:DIP-14_W7.62mm_Socket
- U7: footprint Package_DIP:DIP-16_W7.62mm_LongPads -> rumblesan-standard-parts:DIP-16_W7.62mm_Socket
Connections:
- net +12V: now also R73.1
- net -12V: now also R74.2; no longer R9.2
- net Filter/Input: now also C10.2, R18.2, U2.7
- net Final_Output_Main: now also TP11.1
- net GND: now also R9.2
- net OSC2_LFO_Signal: now also Q9.1 (E), R74.1; no longer Q3.1 (E), R9.1
- net OutputVCA/Input: now also TP10.1
- net Trigger: now also C9.2
- net at C14.2, R33.2, R37.1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: now also TP12.1
- net Filter_LFO_Mod_Ctrl: now reaches J11.4 (Pin_4), RV9.3
- net at J3.1 (Pin_1), R12.1, U3.1: now also C36.2
- net at R10.2, R12.2, U3.2 (-): now also C36.1
- net at U1.4: now also C9.1
- new net: Q3.1 (E), Q9.2 (B), R9.1
- new net: Q9.3 (C), R73.2
Other:
- note added: "Filter Frequency CV Handling"
- note added: "Mixer"
- note added: "Mixer Level Controls"
- note added: "Noise"
- note added: "OSC1"
- note added: "OSC2"
- note added: "Oscillator Frequency Controls"
- note added: "PCB Hardware"
- note added: "Piezo Amplifier"
- moved on the sheet: C12, C13, C15, C8, D1, D2, D3, D4, D5, J1, J10, J11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

Commit message: Further tweaks and layout improvements
Parts:
- removed H1, H2, H3, H4: MountingScrew_M3, MountingHole:MountingHole_3.2mm_M3, symbol Board_Hardware:MountingScrew_M3
- removed H5, H6: Standoff_F-F, symbol Board_Hardware:Standoff_F-F
- C1, C13, C15, C6, C7, C9: Spec (none) -> electrolytic; Tolerance (none) -> 20%; Voltage (none) -> 50v
- C10, C12, C14, C2, C3, C36, C4, C8: Spec (none) -> ceramic C0G; Tolerance (none) -> 5%
- C16: value 1uF (non polarised) -> 1uF; Spec (none) -> electrolytic non polarised; Tolerance (none) -> 20%; Voltage (none) -> 50v
- C5: value 100nF (X7R) -> 100nF; Spec (none) -> ceramic X7R; Tolerance (none) -> 5%
- J10, J4: value Conn_01x04_Male -> Conn_01x04_Header
- J11, J3: value Conn_01x04_Female -> Conn_01x04_Socket
- J12, J18, J2, J26: value AudioJack2_SwitchT -> Eurorack Mono Jack; symbol Connector:AudioJack2_SwitchT -> Eurorack_Hardware:Eurorack Mono Jack; mpn (none) -> WQP-WQP518MA
- J20, J23: value Conn_01x02_Female -> Conn_01x02_Socket
- J21, J22: value Conn_01x02_Male -> Conn_01x02_Header
- J5: value Conn_01x03_Male -> Conn_01x03_Header
- J6, J8: value Conn_01x06_Male -> Conn_01x06_Header
- J7, J9: value Conn_01x06_Female -> Conn_01x06_Socket
- R1, R10, R11, R12, R13, R14, R15, R16, R17, R18, R19, R2, R20, R21, R22, R24, R25, R26, R27, R29, R3, R30, R31, R32, R33, R34, R35, R36, R37, R38, R39, R4, R40, R41, R42, R5, R6, R7, R73, R74, R8, R9: Tolerance (none) -> 1%
- R23: value 82k -> 47k; Tolerance (none) -> 1%
- R28: value 51r -> 47r; Tolerance (none) -> 1%
- RV1: Spec (none) -> single turn
- RV10, RV11, RV7: value 100k -> 100kB
- SW1: value SW_DPDT_x2 -> DPDT; Name (none) -> OSC2 LFO; PartNumber (none) -> MHPS2285
- SW1: value SW_DPDT_x2 -> DPDT; PartNumber (none) -> MHPS2285
- U1: value CD4093B -> CD4093
Connections:
- net GND: now also J2.TN (Tip_normalize); no longer J2.S
- net at J3.2 (Pin_2): now also J2.S (Sleeve); no longer J2.TN
Other:
- note removed: "PCB Hardware"
- moved on the sheet: J2, J26
