File: output-vca.kicad_sch (KiCad schematic)
At the start: 8 parts, among them J27 LevelSelect, U2 TL072, U7 LM13700

Commit message: Updating after tweaks and project improvements
Parts:
- J27: value LevelSelect -> Conn_01x03_Male; Name (none) -> Output Level Select
- R68, R69, R70: footprint Rumblesan_Footprints:Resistor_THT_L6.3mm_D2.5mm_P10.16mm_Horizontal -> rumblesan-standard-parts:R_Axial_DIN0207_L6.3mm_D2.5mm_P10.16mm_Horizontal
- R71: value 18k -> 33k; footprint Rumblesan_Footprints:Resistor_THT_L6.3mm_D2.5mm_P10.16mm_Horizontal -> rumblesan-standard-parts:R_Axial_DIN0207_L6.3mm_D2.5mm_P10.16mm_Horizontal
- R72: value 4k7 -> 10k; footprint Rumblesan_Footprints:Resistor_THT_L6.3mm_D2.5mm_P10.16mm_Horizontal -> rumblesan-standard-parts:R_Axial_DIN0207_L6.3mm_D2.5mm_P10.16mm_Horizontal
- U2: footprint Package_DIP:DIP-8_W7.62mm_LongPads -> rumblesan-standard-parts:DIP-8_W7.62mm_Socket
- U7: footprint Package_DIP:DIP-16_W7.62mm_LongPads -> rumblesan-standard-parts:DIP-16_W7.62mm_Socket
Connections:
- net at U2.2 (-), U7.12: now also J27.2 (Pin_2); no longer J27.3 (Pin_3)
- net at R72.1: now also J27.3 (Pin_3); no longer J27.2 (Pin_2)
Other:
- title: (none) -> Magnum Percussion Instrument
- moved on the sheet: J27
Changed lines of the file:
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@@
 (kicad_sch (version 20211123) (generator eeschema)
   (paper "A4")
+  (title_block
+    (title "Magnum Percussion Instrument")
+    (date "2022-06-15")
+    (rev "r03")
+    (comment 2 "creativecommons.org/licenses/by/4.0/")
+    (comment 3 "License: CC BY 4.0")
+    (comment 4 "Author: Guy John")
+  )
+  (junction (at 167.64 72.39) (diameter 0) (color 0 0 0 0)
+  )
   (junction (at 167.64 88.9) (diameter 0) (color 0 0 0 0)
-  )
-  (junction (at 167.64 72.39) (diameter 0) (color 0 0 0 0)
   )
   (junction (at 147.32 86.36) (diameter 0) (color 0 0 0 0)
@@
     (stroke (width 0) (type default) (color 0 0 0 0))
   )
-  (wire (pts (xy 146.05 74.93) (xy 147.32 74.93))
-    (stroke (width 0) (type default) (color 0 0 0 0))
-  )
-  (wire (pts (xy 167.64 88.9) (xy 167.64 72.39))
-    (stroke (width 0) (type default) (color 0 0 0 0))
-  )
   (wire (pts (xy 167.64 67.31) (xy 158.75 67.31))
     (stroke (width 0) (type default) (color 0 0 0 0))
@@
     (stroke (width 0) (type default) (color 0 0 0 0))
   )
+  (wire (pts (xy 149.86 91.44) (xy 148.59 91.44))
+    (stroke (width 0) (type default) (color 0 0 0 0))
+  )
+  (wire (pts (xy 167.64 67.31) (xy 167.64 72.39))
+    (stroke (width 0) (type default) (color 0 0 0 0))
+  )
+  (wire (pts (xy 147.32 69.85) (xy 146.05 69.85))
+    (stroke (width 0) (type default) (color 0 0 0 0))
+  )
+  (wire (pts (xy 148.59 91.44) (xy 148.59 92.71))
+    (stroke (width 0) (type default) (color 0 0 0 0))
+  )
+  (wire (pts (xy 137.16 88.9) (xy 134.62 88.9))
+    (stroke (width 0) (type default) (color 0 0 0 0))
+  )
+  (wire (pts (xy 147.32 86.36) (xy 149.86 86.36))
+    (stroke (width 0) (type default) (color 0 0 0 0))
+  )
+  (wire (pts (xy 146.05 67.31) (xy 151.13 67.31))
+    (stroke (width 0) (type default) (color 0 0 0 0))
+  )
+  (wire (pts (xy 91.44 83.82) (xy 95.25 83.82))
+    (stroke (width 0) (type default) (color 0 0 0 0))
+  )
+  (wire (pts (xy 119.38 88.9) (xy 115.57 88.9))
+    (stroke (width 0) (type default) (color 0 0 0 0))
+  )
+  (wire (pts (xy 106.68 92.71) (xy 106.68 83.82))
+    (stroke (width 0) (type default) (color 0 0 0 0))
+  )
+  (wire (pts (xy 106.68 100.33) (xy 106.68 102.87))
+    (stroke (width 0) (type default) (color 0 0 0 0))
+  )
+  (wire (pts (xy 158.75 72.39) (xy 167.64 72.39))
+    (stroke (width 0) (type default) (color 0 0 0 0))
+  )
+  (wire (pts (xy 167.64 72.39) (xy 167.64 88.9))
+    (stroke (width 0) (type default) (color 0 0 0 0))
+  )
+  (wire (pts (xy 137.16 88.9) (xy 137.16 115.57))
+    (stroke (width 0) (type default) (color 0 0 0 0))
+  )
   (wire (pts (xy 146.05 72.39) (xy 151.13 72.39))
     (stroke (width 0) (type default) (color 0 0 0 0))
   )
-  (wire (pts (xy 149.86 91.44) (xy 148.59 91.44))
-    (stroke (width 0) (type default) (color 0 0 0 0))
-  )
-  (wire (pts (xy 167.64 72.39) (xy 167.64 67.31))
-    (stroke (width 0) (type default) (color 0 0 0 0))
-  )
-  (wire (pts (xy 148.59 91.44) (xy 148.59 92.71))
-    (stroke (width 0) (type default) (color 0 0 0 0))
-  )
-  (wire (pts (xy 137.16 88.9) (xy 134.62 88.9))
-    (stroke (width 0) (type default) (color 0 0 0 0))
-  )
-  (wire (pts (xy 148.59 69.85) (xy 148.59 67.31))
-    (stroke (width 0) (type default) (color 0 0 0 0))
-  )
-  (wire (pts (xy 146.05 69.85) (xy 148.59 69.85))
-    (stroke (width 0) (type default) (color 0 0 0 0))
-  )
-  (wire (pts (xy 147.32 86.36) (xy 149.86 86.36))
-    (stroke (width 0) (type default) (color 0 0 0 0))
-  )
-  (wire (pts (xy 148.59 67.31) (xy 151.13 67.31))
-    (stroke (width 0) (type default) (color 0 0 0 0))
-  )
-  (wire (pts (xy 91.44 83.82) (xy 95.25 83.82))
-    (stroke (width 0) (type default) (color 0 0 0 0))
-  )
-  (wire (pts (xy 119.38 88.9) (xy 115.57 88.9))
-    (stroke (width 0) (type default) (color 0 0 0 0))
-  )
-  (wire (pts (xy 106.68 92.71) (xy 106.68 83.82))
-    (stroke (width 0) (type default) (color 0 0 0 0))
-  )
-  (wire (pts (xy 106.68 100.33) (xy 106.68 102.87))
-    (stroke (width 0) (type default) (color 0 0 0 0))
-  )
-  (wire (pts (xy 137.16 88.9) (xy 137.16 115.57))
-    (stroke (width 0) (type default) (color 0 0 0 0))
-  )
   (wire (pts (xy 115.57 100.33) (xy 115.57 102.87))
     (stroke (width 0) (type default) (color 0 0 0 0))
@@
     (stroke (width 0) (type default) (color 0 0 0 0))
   )
-  (wire (pts (xy 167.64 72.39) (xy 158.75 72.39))
-    (stroke (width 0) (type default) (color 0 0 0 0))
-  )
   (wire (pts (xy 106.68 83.82) (xy 119.38 83.82))
     (stroke (width 0) (type default) (color 0 0 0 0))
   )
-  (wire (pts (xy 147.32 74.93) (xy 147.32 86.36))
+  (wire (pts (xy 147.32 69.85) (xy 147.32 86.36))
     (stroke (width 0) (type default) (color 0 0 0 0))
   )
@@
     (in_bom yes) (on_board yes) (fields_autoplaced)
     (property "Reference" "R71" (id 0) (at 154.94 62.3275 90))
-    (property "Value" "18k" (id 1) (at 154.94 65.1026 90))
-    (property "Footprint" "Rumblesan_Footprints:Resistor_THT_L6.3mm_D2.5mm_P10.16mm_Horizontal" (id 2) (at 154.94 69.088 90)
+    (property "Value" "33k" (id 1) (at 154.94 65.1026 90))
+    (property "Footprint" "rumblesan-standard-parts:R_Axial_DIN0207_L6.3mm_D2.5mm_P10.16mm_Horizontal" (id 2) (at 154.94 69.088 90)
       (effects (font (size 1.27 1.27)) hide)
     )
@@
     (property "Reference" "U7" (id 0) (at 127 77.3135 0))
     (property "Value" "LM13700" (id 1) (at 127 80.0886 0))
-    (property "Footprint" "Package_DIP:DIP-16_W7.62mm_LongPads" (id 2) (at 119.38 85.725 0)
+    (property "Footprint" "rumblesan-standard-parts:DIP-16_W7.62mm_Socket" (id 2) (at 119.38 85.725 0)
       (effects (font (size 1.27 1.27)) hide)
     )
@@
     (pin "16")
   )
-  (symbol (lib_id "Connector:Conn_01x03_Male") (at 140.97 72.39 0) (unit 1)
-    (in_bom yes) (on_board yes) (fields_autoplaced)
-    (property "Reference" "J27" (id 0) (at 141.605 65.8073 0))
-    (property "Value" "LevelSelect" (id 1) (at 141.605 68.5824 0))
-    (property "Footprint" "Connector_PinHeader_2.54mm:PinHeader_1x03_P2.54mm_Vertical" (id 2) (at 140.97 72.39 0)
-      (effects (font (size 1.27 1.27)) hide)
-    )
-    (property "Datasheet" "~" (id 3) (at 140.97 72.39 0)
-      (effects (font (size 1.27 1.27)) hide)
-    )
+  (symbol (lib_id "Connector:Conn_01x03_Male") (at 140.97 69.85 0) (unit 1)
+    (in_bom yes) (on_board yes)
+    (property "Reference" "J27" (id 0) (at 140.97 74.93 0))
+    (property "Value" "Conn_01x03_Male" (id 1) (at 141.605 66.0424 0)
+      (effects (font (size 1.27 1.27)) hide)
+    )
+    (property "Footprint" "Connector_PinHeader_2.54mm:PinHeader_1x03_P2.54mm_Vertical" (id 2) (at 140.97 69.85 0)
+      (effects (font (size 1.27 1.27)) hide)
+    )
+    (property "Datasheet" "~" (id 3) (at 140.97 69.85 0)
+      (effects (font (size 1.27 1.27)) hide)
+    )
+    (property "Name" "Output Level Select" (id 4) (at 140.97 63.5 0))
     (pin "1")
     (pin "2")
@@
     (in_bom yes) (on_board yes)
     (property "Reference" "R72" (id 0) (at 154.94 74.93 90))
-    (property "Value" "4k7" (id 1) (at 154.94 70.1826 90))
-    (property "Footprint" "Rumblesan_Footprints:Resistor_THT_L6.3mm_D2.5mm_P10.16mm_Horizontal" (id 2) (at 154.94 74.168 90)
+    (property "Value" "10k" (id 1) (at 154.94 70.1826 90))
+    (property "Footprint" "rumblesan-standard-parts:R_Axial_DIN0207_L6.3mm_D2.5mm_P10.16mm_Horizontal" (id 2) (at 154.94 74.168 90)
       (effects (font (size 1.27 1.27)) hide)
     )
@@
     (property "Reference" "U2" (id 0) (at 157.48 79.8535 0))
     (property "Value" "TL072" (id 1) (at 157.48 82.6286 0))
-    (property "Footprint" "Package_DIP:DIP-8_W7.62mm_LongPads" (id 2) (at 157.48 88.9 0)
+    (property "Footprint" "rumblesan-standard-parts:DIP-8_W7.62mm_Socket" (id 2) (at 157.48 88.9 0)
       (effects (font (size 1.27 1.27)) hide)
     )
@@
     (property "Reference" "R68" (id 0) (at 99.06 78.8375 90))
     (property "Value" "100k" (id 1) (at 99.06 81.6126 90))
-    (property "Footprint" "Rumblesan_Footprints:Resistor_THT_L6.3mm_D2.5mm_P10.16mm_Horizontal" (id 2) (at 99.06 85.598 90)
+    (property "Footprint" "rumblesan-standard-parts:R_Axial_DIN0207_L6.3mm_D2.5mm_P10.16mm_Horizontal" (id 2) (at 99.06 85.598 90)
       (effects (font (size 1.27 1.27)) hide)
     )
@@
       (effects (font (size 1.27 1.27)) (justify left))
     )
-    (property "Footprint" "Rumblesan_Footprints:Resistor_THT_L6.3mm_D2.5mm_P10.16mm_Horizontal" (id 2) (at 104.902 96.52 90)
+    (property "Footprint" "rumblesan-standard-parts:R_Axial_DIN0207_L6.3mm_D2.5mm_P10.16mm_Horizontal" (id 2) (at 104.902 96.52 90)
       (effects (font (size 1.27 1.27)) hide)
     )
@@
       (effects (font (size 1.27 1.27)) (justify left))
     )
-    (property "Footprint" "Rumblesan_Footprints:Resistor_THT_L6.3mm_D2.5mm_P10.16mm_Horizontal" (id 2) (at 113.792 96.52 90)
+    (property "Footprint" "rumblesan-standard-parts:R_Axial_DIN0207_L6.3mm_D2.5mm_P10.16mm_Horizontal" (id 2) (at 113.792 96.52 90)
       (effects (font (size 1.27 1.27)) hide)
     )
@@
     (property "Reference" "U7" (id 0) (at 182.88 48.2399 0))
     (property "Value" "LM13700" (id 1) (at 182.88 51.015 0))
-    (property "Footprint" "Package_DIP:DIP-16_W7.62mm_LongPads" (id 2) (at 177.8 56.515 0)
-      (effects (font (size 1.27 1.27)) hide)
-    )
+    (property "Footprint" "rumblesan-standard-parts:DIP-16_W7.62mm_Socket" (id 2) (at 177.8 56.515 0)
+      (effects (font (size 1.27 1.27)) hide)
+    )

Commit message: Further tweaks and layout improvements
Parts:
- J27: value Conn_01x03_Male -> Conn_01x03_Header
- R68, R69, R70, R71, R72: Tolerance (none) -> 1%
Changed lines of the file:
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@@
+      (effects (font (size 1.27 1.27)) hide)
+    )
+    (property "Tolerance" "1%" (id 4) (at 154.94 67.31 0)
       (effects (font (size 1.27 1.27)) hide)
     )
@@
     (pin "15")
     (pin "16")
+    (pin "10")
+    (pin "9")
+    (pin "1")
+    (pin "2")
+    (pin "3")
+    (pin "4")
+    (pin "5")
+    (pin "7")
+    (pin "8")
+    (pin "11")
+    (pin "6")
   )
   (symbol (lib_id "Connector:Conn_01x03_Male") (at 140.97 69.85 0) (unit 1)
     (in_bom yes) (on_board yes)
     (property "Reference" "J27" (id 0) (at 140.97 74.93 0))
-    (property "Value" "Conn_01x03_Male" (id 1) (at 141.605 66.0424 0)
+    (property "Value" "Conn_01x03_Header" (id 1) (at 141.605 66.0424 0)
       (effects (font (size 1.27 1.27)) hide)
     )
@@
       (effects (font (size 1.27 1.27)) hide)
     )
+    (property "Tolerance" "1%" (id 4) (at 154.94 72.39 0)
+      (effects (font (size 1.27 1.27)) hide)
+    )
     (pin "1")
     (pin "2")
@@
     (pin "2")
     (pin "3")
+    (pin "5")
+    (pin "6")
+    (pin "7")
+    (pin "4")
+    (pin "8")
   )
   (symbol (lib_id "power:GND") (at 115.57 102.87 0) (unit 1)
@@
       (effects (font (size 1.27 1.27)) hide)
     )
+    (property "Tolerance" "1%" (id 4) (at 99.06 83.82 0)
+      (effects (font (size 1.27 1.27)) hide)
+    )
     (pin "1")
     (pin "2")
@@
     )
     (property "Datasheet" "~" (id 3) (at 106.68 96.52 0)
+      (effects (font (size 1.27 1.27)) hide)
+    )
+    (property "Tolerance" "1%" (id 4) (at 106.68 96.52 0)
       (effects (font (size 1.27 1.27)) hide)
     )
@@
       (effects (font (size 1.27 1.27)) hide)
     )
+    (property "Tolerance" "1%" (id 4) (at 115.57 96.52 0)
+      (effects (font (size 1.27 1.27)) hide)
+    )
     (pin "1")
     (pin "2")
@@
       (effects (font (size 1.27 1.27)) hide)
     )
+    (pin "12")
+    (pin "13")
+    (pin "14")
+    (pin "15")
+    (pin "16")
     (pin "10")
     (pin "9")
+    (pin "1")
+    (pin "2")
+    (pin "3")
+    (pin "4")
+    (pin "5")
+    (pin "7")
+    (pin "8")
+    (pin "11")
+    (pin "6")
   )
   (symbol (lib_id "power:GND") (at 106.68 102.87 0) (unit 1)
