File: power.kicad_sch (KiCad schematic)
At the start: 27 parts, among them J28 Eurorack_Power_Small, J29 POWER_CTRL, J30 POWER_MAIN, U1 HEF4093B, U2 TL072, U3 TL072, U4 TL074, U5 LM13700, U6 LM13700, U7 LM13700

Commit message: Updating after tweaks and project improvements
Parts:
- C21, C22: footprint Capacitor_THT:CP_Radial_D5.0mm_P2.50mm -> rumblesan-standard-parts:CP_Radial_D5.0mm_P2.00mm
- C23, C24, C25, C26, C27, C28, C29, C30, C31, C32, C33, C34, C35: footprint Rumblesan_Footprints:C_Rect_L7.0mm_W3.5mm_P5.00mm -> rumblesan-standard-parts:C_Rect_L7.0mm_W3.5mm_P5.00mm
- D7, D8: footprint Rumblesan_Footprints:D_DO-35_SOD27_P7.62mm_Horizontal -> rumblesan-standard-parts:D_DO-41_SOD81_P10.16mm_Horizontal
- J28: footprint EurorackBasics:Eurorack_PowerHeader_2x05_P2.54mm_Shrouded -> eurorack-power:Eurorack_PowerHeader_2x05_P2.54mm_Shrouded
- U1: value HEF4093B -> CD4093B; footprint Package_DIP:DIP-14_W7.62mm_LongPads -> rumblesan-standard-parts:DIP-14_W7.62mm_Socket
- U2, U3: footprint Package_DIP:DIP-8_W7.62mm_LongPads -> rumblesan-standard-parts:DIP-8_W7.62mm_Socket
- U4: footprint Package_DIP:DIP-14_W7.62mm_LongPads -> rumblesan-standard-parts:DIP-14_W7.62mm_Socket
- U5, U6, U7: footprint Package_DIP:DIP-16_W7.62mm_LongPads -> rumblesan-standard-parts:DIP-16_W7.62mm_Socket
Other:
- title: (none) -> Magnum Percussion Instrument
Changed lines of the file:
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@@
 (kicad_sch (version 20211123) (generator eeschema)
   (paper "A4")
+  (title_block
+    (title "Magnum Percussion Instrument")
+    (date "2022-06-15")
+    (rev "r03")
+    (comment 2 "creativecommons.org/licenses/by/4.0/")
+    (comment 3 "License: CC BY 4.0")
+    (comment 4 "Author: Guy John")
+  )
   (junction (at 199.39 43.18) (diameter 0) (color 0 0 0 0)
   )
@@
       (effects (font (size 1.27 1.27)) (justify left))
     )
-    (property "Footprint" "Capacitor_THT:CP_Radial_D5.0mm_P2.50mm" (id 2) (at 68.2752 72.39 0)
+    (property "Footprint" "rumblesan-standard-parts:CP_Radial_D5.0mm_P2.00mm" (id 2) (at 68.2752 72.39 0)
       (effects (font (size 1.27 1.27)) hide)
     )
@@
       (effects (font (size 1.27 1.27)) (justify left))
     )
-    (property "Footprint" "Rumblesan_Footprints:C_Rect_L7.0mm_W3.5mm_P5.00mm" (id 2) (at 113.9952 76.2 0)
+    (property "Footprint" "rumblesan-standard-parts:C_Rect_L7.0mm_W3.5mm_P5.00mm" (id 2) (at 113.9952 76.2 0)
       (effects (font (size 1.27 1.27)) hide)
     )
@@
       (effects (font (size 1.27 1.27)) (justify left))
     )
-    (property "Footprint" "Rumblesan_Footprints:C_Rect_L7.0mm_W3.5mm_P5.00mm" (id 2) (at 122.8852 76.2 0)
+    (property "Footprint" "rumblesan-standard-parts:C_Rect_L7.0mm_W3.5mm_P5.00mm" (id 2) (at 122.8852 76.2 0)
       (effects (font (size 1.27 1.27)) hide)
     )
@@
       (effects (font (size 1.27 1.27)) (justify left))
     )
-    (property "Footprint" "Package_DIP:DIP-8_W7.62mm_LongPads" (id 2) (at 111.76 46.99 0)
+    (property "Footprint" "rumblesan-standard-parts:DIP-8_W7.62mm_Socket" (id 2) (at 111.76 46.99 0)
       (effects (font (size 1.27 1.27)) hide)
     )
@@
     (property "Reference" "D8" (id 0) (at 60.96 73.5035 0))
     (property "Value" "1N5818" (id 1) (at 60.96 76.2786 0))
-    (property "Footprint" "Rumblesan_Footprints:D_DO-35_SOD27_P7.62mm_Horizontal" (id 2) (at 60.96 78.74 0)
+    (property "Footprint" "rumblesan-standard-parts:D_DO-41_SOD81_P10.16mm_Horizontal" (id 2) (at 60.96 78.74 0)
       (effects (font (size 1.27 1.27)) hide)
     )
@@
       (effects (font (size 1.27 1.27)) (justify left))
     )
-    (property "Footprint" "Rumblesan_Footprints:C_Rect_L7.0mm_W3.5mm_P5.00mm" (id 2) (at 149.5552 86.36 0)
+    (property "Footprint" "rumblesan-standard-parts:C_Rect_L7.0mm_W3.5mm_P5.00mm" (id 2) (at 149.5552 86.36 0)
       (effects (font (size 1.27 1.27)) hide)
     )
@@
     (property "Reference" "J28" (id 0) (at 47.625 50.0593 0))
     (property "Value" "Eurorack_Power_Small" (id 1) (at 43.18 59.69 90))
-    (property "Footprint" "EurorackBasics:Eurorack_PowerHeader_2x05_P2.54mm_Shrouded" (id 2) (at 48.26 60.96 0)
+    (property "Footprint" "eurorack-power:Eurorack_PowerHeader_2x05_P2.54mm_Shrouded" (id 2) (at 48.26 60.96 0)
       (effects (font (size 1.27 1.27)) hide)
     )
@@
       (effects (font (size 1.27 1.27)) (justify left))
     )
-    (property "Footprint" "Package_DIP:DIP-16_W7.62mm_LongPads" (id 2) (at 134.62 46.355 0)
+    (property "Footprint" "rumblesan-standard-parts:DIP-16_W7.62mm_Socket" (id 2) (at 134.62 46.355 0)
       (effects (font (size 1.27 1.27)) hide)
     )
@@
       (effects (font (size 1.27 1.27)) (justify left))
     )
-    (property "Footprint" "Rumblesan_Footprints:C_Rect_L7.0mm_W3.5mm_P5.00mm" (id 2) (at 140.6652 86.36 0)
+    (property "Footprint" "rumblesan-standard-parts:C_Rect_L7.0mm_W3.5mm_P5.00mm" (id 2) (at 140.6652 86.36 0)
       (effects (font (size 1.27 1.27)) hide)
     )
@@
       (effects (font (size 1.27 1.27)) (justify left))
     )
-    (property "Footprint" "Capacitor_THT:CP_Radial_D5.0mm_P2.50mm" (id 2) (at 68.2752 53.34 0)
+    (property "Footprint" "rumblesan-standard-parts:CP_Radial_D5.0mm_P2.00mm" (id 2) (at 68.2752 53.34 0)
       (effects (font (size 1.27 1.27)) hide)
     )
@@
     (property "Reference" "D7" (id 0) (at 60.96 35.4035 0))
     (property "Value" "1N5818" (id 1) (at 60.96 38.1786 0))
-    (property "Footprint" "Rumblesan_Footprints:D_DO-35_SOD27_P7.62mm_Horizontal" (id 2) (at 60.96 40.64 0)
+    (property "Footprint" "rumblesan-standard-parts:D_DO-41_SOD81_P10.16mm_Horizontal" (id 2) (at 60.96 40.64 0)
       (effects (font (size 1.27 1.27)) hide)
     )
@@
       (effects (font (size 1.27 1.27)) (justify left))
     )
-    (property "Footprint" "Rumblesan_Footprints:C_Rect_L7.0mm_W3.5mm_P5.00mm" (id 2) (at 113.9952 86.36 0)
+    (property "Footprint" "rumblesan-standard-parts:C_Rect_L7.0mm_W3.5mm_P5.00mm" (id 2) (at 113.9952 86.36 0)
       (effects (font (size 1.27 1.27)) hide)
     )
@@
       (effects (font (size 1.27 1.27)) (justify left))
     )
-    (property "Footprint" "Rumblesan_Footprints:C_Rect_L7.0mm_W3.5mm_P5.00mm" (id 2) (at 140.6652 76.2 0)
+    (property "Footprint" "rumblesan-standard-parts:C_Rect_L7.0mm_W3.5mm_P5.00mm" (id 2) (at 140.6652 76.2 0)
       (effects (font (size 1.27 1.27)) hide)
     )
@@
       (effects (font (size 1.27 1.27)) (justify left))
     )
-    (property "Value" "HEF4093B" (id 1) (at 207.01 67.31 90)
-      (effects (font (size 1.27 1.27)) (justify left))
-    )
-    (property "Footprint" "Package_DIP:DIP-14_W7.62mm_LongPads" (id 2) (at 199.39 57.15 0)
-      (effects (font (size 1.27 1.27)) hide)
-    )
-    (property "Datasheet" "https://assets.nexperia.com/documents/data-sheet/HEF4093B.pdf" (id 3) (at 199.39 57.15 0)
+    (property "Value" "CD4093B" (id 1) (at 207.01 67.31 90)
+      (effects (font (size 1.27 1.27)) (justify left))
+    )
+    (property "Footprint" "rumblesan-standard-parts:DIP-14_W7.62mm_Socket" (id 2) (at 199.39 57.15 0)
+      (effects (font (size 1.27 1.27)) hide)
+    )
+    (property "Datasheet" "https://www.ti.com/lit/ds/symlink/cd4093b.pdf" (id 3) (at 199.39 57.15 0)
       (effects (font (size 1.27 1.27)) hide)
     )
@@
       (effects (font (size 1.27 1.27)) (justify left))
     )
-    (property "Footprint" "Rumblesan_Footprints:C_Rect_L7.0mm_W3.5mm_P5.00mm" (id 2) (at 131.7752 76.2 0)
+    (property "Footprint" "rumblesan-standard-parts:C_Rect_L7.0mm_W3.5mm_P5.00mm" (id 2) (at 131.7752 76.2 0)
       (effects (font (size 1.27 1.27)) hide)
     )
@@
       (effects (font (size 1.27 1.27)) (justify left))
     )
-    (property "Footprint" "Package_DIP:DIP-8_W7.62mm_LongPads" (id 2) (at 104.14 46.99 0)
+    (property "Footprint" "rumblesan-standard-parts:DIP-8_W7.62mm_Socket" (id 2) (at 104.14 46.99 0)
       (effects (font (size 1.27 1.27)) hide)
     )
@@
       (effects (font (size 1.27 1.27)) (justify left))
     )
-    (property "Footprint" "Package_DIP:DIP-16_W7.62mm_LongPads" (id 2) (at 123.19 46.355 0)
+    (property "Footprint" "rumblesan-standard-parts:DIP-16_W7.62mm_Socket" (id 2) (at 123.19 46.355 0)
       (effects (font (size 1.27 1.27)) hide)
     )
@@
       (effects (font (size 1.27 1.27)) (justify left))
     )
-    (property "Footprint" "Rumblesan_Footprints:C_Rect_L7.0mm_W3.5mm_P5.00mm" (id 2) (at 122.8852 86.36 0)
+    (property "Footprint" "rumblesan-standard-parts:C_Rect_L7.0mm_W3.5mm_P5.00mm" (id 2) (at 122.8852 86.36 0)
       (effects (font (size 1.27 1.27)) hide)
     )
@@
       (effects (font (size 1.27 1.27)) (justify left))
     )
-    (property "Footprint" "Rumblesan_Footprints:C_Rect_L7.0mm_W3.5mm_P5.00mm" (id 2) (at 190.1952 60.96 0)
+    (property "Footprint" "rumblesan-standard-parts:C_Rect_L7.0mm_W3.5mm_P5.00mm" (id 2) (at 190.1952 60.96 0)
       (effects (font (size 1.27 1.27)) hide)
     )
@@
       (effects (font (size 1.27 1.27)) (justify left))
     )
-    (property "Footprint" "Rumblesan_Footprints:C_Rect_L7.0mm_W3.5mm_P5.00mm" (id 2) (at 149.5552 76.2 0)
+    (property "Footprint" "rumblesan-standard-parts:C_Rect_L7.0mm_W3.5mm_P5.00mm" (id 2) (at 149.5552 76.2 0)
       (effects (font (size 1.27 1.27)) hide)
     )
@@
       (effects (font (size 1.27 1.27)) (justify left))
     )
-    (property "Footprint" "Package_DIP:DIP-14_W7.62mm_LongPads" (id 2) (at 95.25 44.45 0)
+    (property "Footprint" "rumblesan-standard-parts:DIP-14_W7.62mm_Socket" (id 2) (at 95.25 44.45 0)
       (effects (font (size 1.27 1.27)) hide)
     )
@@
       (effects (font (size 1.27 1.27)) (justify left))
     )
-    (property "Footprint" "Rumblesan_Footprints:C_Rect_L7.0mm_W3.5mm_P5.00mm" (id 2) (at 105.1052 76.2 0)
+    (property "Footprint" "rumblesan-standard-parts:C_Rect_L7.0mm_W3.5mm_P5.00mm" (id 2) (at 105.1052 76.2 0)
       (effects (font (size 1.27 1.27)) hide)
     )
@@
       (effects (font (size 1.27 1.27)) (justify left))
     )
-    (property "Footprint" "Rumblesan_Footprints:C_Rect_L7.0mm_W3.5mm_P5.00mm" (id 2) (at 105.1052 86.36 0)
+    (property "Footprint" "rumblesan-standard-parts:C_Rect_L7.0mm_W3.5mm_P5.00mm" (id 2) (at 105.1052 86.36 0)
       (effects (font (size 1.27 1.27)) hide)
     )
@@
       (effects (font (size 1.27 1.27)) (justify left))
     )
-    (property "Footprint" "Package_DIP:DIP-16_W7.62mm_LongPads" (id 2) (at 111.76 46.355 0)
+    (property "Footprint" "rumblesan-standard-parts:DIP-16_W7.62mm_Socket" (id 2) (at 111.76 46.355 0)
       (effects (font (size 1.27 1.27)) hide)
     )
@@
       (effects (font (size 1.27 1.27)) (justify left))
     )
-    (property "Footprint" "Rumblesan_Footprints:C_Rect_L7.0mm_W3.5mm_P5.00mm" (id 2) (at 131.7752 86.36 0)
-      (effects (font (size 1.27 1.27)) hide)
-    )
+    (property "Footprint" "rumblesan-standard-parts:C_Rect_L7.0mm_W3.5mm_P5.00mm" (id 2) (at 131.7752 86.36 0)
+      (effects (font (size 1.27 1.27)) hide)
+    )

Commit message: Further tweaks and layout improvements
Parts:
- C21, C22: Spec (none) -> electrolytic; Tolerance (none) -> 20%; Voltage (none) -> 50v
- C23, C24, C25, C26, C27, C28, C29, C30, C31, C32, C33, C34, C35: value 100nF (X7R) -> 100nF; Spec (none) -> ceramic X7R; Tolerance (none) -> 5%
- J28: value Eurorack_Power_Small -> Eurorack Power Small; symbol Eurorack_Hardware:Eurorack_Power_Small -> Eurorack_Hardware:Eurorack Power Small
- J29: value POWER_CTRL -> Conn_01x04_Socket; Name (none) -> Power Header Ctrl
- J30: value POWER_MAIN -> Conn_01x04_Header; Name (none) -> Power Header Main
- U1: value CD4093B -> CD4093
