File: kicad/magnum-drum-synth.kicad_sch (KiCad schematic)
At the start: 129 parts, among them J10 Conn_01x04_Header, J11 Conn_01x04_Socket, J12 Eurorack Mono Jack, J18 Eurorack Mono Jack, J2 Eurorack Mono Jack, J20 Conn_01x02_Socket, J21 Conn_01x02_Header, J22 Conn_01x02_Header, J23 Conn_01x02_Socket, J26 Eurorack Mono Jack, J3 Conn_01x04_Socket, J4 Conn_01x04_Header, J5 Conn_01x03_Header, J6 Conn_01x06_Header, J7 Conn_01x06_Socket, J8 Conn_01x06_Header, J9 Conn_01x06_Socket, Q1 2N3904, Q2 2N3904, Q3 2N3904, Q4 2N3904, Q5 2N3904, Q6 2N3906, Q7 2N3906, Q8 2N3906, Q9 2N3906, SW1 DPDT, U1 CD4093, U2 TL072, U3 TL074, U4 TL074, U7 LM13700

Commit message: Move decay env CV summing to front board
Parts:
- removed J22: Conn_01x02_Header, Connector_PinHeader_2.54mm:PinHeader_1x02_P2.54mm_Vertical, symbol Connector:Conn_01x02_Male
- removed J23: Conn_01x02_Socket, Connector_PinSocket_2.54mm:PinSocket_1x02_P2.54mm_Vertical, symbol Connector:Conn_01x02_Female
Connections:
- net Res_Amount: now also J6.5 (Pin_5)
- net Res_Amount_Ctrl: now also J7.5 (Pin_5)
- net Res_Top: now also J6.6 (Pin_6)
- net Res_Top_Ctrl: now also J7.6 (Pin_6)
- net at C14.1, R27.1, R30.2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: now also U3.6 (-); no longer U4.2 (-)
- net AMP_DECAY_CV_MIX_CTRL: now reaches U3.7
- net AMP_DECAY_CV_MIX_CTRL: now also C14.2, J20.1 (Pin_1), R33.2; no longer U3.6 (-)
- net AMP_DECAY_CTRL: no longer names the net of R25.1, RV10.2
- net AMP_DECAY_CTRL: now also R27.2; no longer J20.2 (Pin_2)
- net AMP_DECAY_CV_CTRL: no longer names the net of J18.T (Tip)
- net AMP_DECAY_CV_CTRL: now also R30.1; no longer J20.1 (Pin_1)
- net AMP_DECAY_CV_MAIN renamed AMP_DECAY_CV_MIX_MAIN
- net AMP_DECAY_CV_MIX_MAIN: now also R37.1, TP12.1; no longer R30.1
- net AMP_DECAY_MAIN: no longer names the net of J21.2 (Pin_2)
- net AMP_DECAY_MAIN: no longer R27.2
- new net: U4.1, U4.2 (-)
- no-connect marks 13 -> 11
Other:
- moved on the sheet: C14, J18, J21, R25, R27, R30, R31, R33, RV10, U3B, U4A

Commit message: slimlining opamp count and more moving around
Parts:
- removed J20: Conn_01x02_Socket, Connector_PinSocket_2.54mm:PinSocket_1x02_P2.54mm_Vertical, symbol Connector:Conn_01x02_Female
- removed J21: Conn_01x02_Header, Connector_PinHeader_2.54mm:PinHeader_1x02_P2.54mm_Vertical, symbol Connector:Conn_01x02_Male
- removed U2: TL072, rumblesan-standard-parts:DIP-8_W7.62mm_Socket, symbol Amplifier_Operational:TL072
- removed unit 1 of U4
- added R76: 47r, rumblesan-standard-parts:R_Axial_DIN0207_L6.3mm_D2.5mm_P10.16mm_Horizontal, symbol Device:R
Connections:
- net PIEZO_NORMAL_CTRL is gone; now on net PIEZO_CTRL: J2.TN (Tip_normalize), J3.2 (Pin_2)
- net AMP_DECAY_CV_MIX_CTRL: now also J3.1 (Pin_1)
- net AMP_DECAY_CV_MIX_MAIN: now also J4.1 (Pin_1)
- net PIEZO_CTRL: no longer J3.1 (Pin_1)
- net PIEZO_MAIN: now also J4.2 (Pin_2); no longer J4.1 (Pin_1)
- net Trigger: now also U4.13 (-), U4.14, R76.1; no longer C9.2, R14.1, TP5.1, U1.1, U1.2, U4.12 (+)
- net at C9.1, U1.4: now also TP5.1, U4.12 (+)
- net Filter_Env renamed FILTER_ENV_MOD_MAIN
- net Filter_Env_Decay renamed FILTER_ENV_DECAY_MAIN
- net Filter_Env_Decay_Ctrl renamed FILTER_ENV_DECAY_CTRL
- net Filter_Env_Mod_Ctrl renamed FILTER_ENV_MOD_CTRL
- net Filter_LFO_Mod_Ctrl renamed OSC2_FILTER_MOD_CTRL
- net Freq_Control_Ctrl renamed FILTER_FREQ_CV_CTRL
- net Freq_Control_Main renamed FILTER_FREQ_CV_MAIN
- net Noise_Signal renamed NOISE_SIGNAL_MAIN
- net Noise_Signal_Ctrl renamed NOISE_SIGNAL_CTRL
- net OSC1_Freq_L renamed OSC1_FREQ_L_MAIN
- net OSC1_Freq_L_Ctrl renamed OSC1_FREQ_L_CTRL
- net OSC1_Freq_R renamed OSC1_FREQ_R_MAIN
- net OSC1_Freq_R_Ctrl renamed OSC1_FREQ_R_CTRL
- net OSC1_Signal renamed OSC1_SIGNAL_MAIN
- net OSC1_Signal_Ctrl renamed OSC1_SIGNAL_CTRL
- net OSC2_Freq_L renamed OSC2_FREQ_L_MAIN
- net OSC2_Freq_L_Ctrl renamed OSC2_FREQ_L_CTRL
- net OSC2_Freq_R renamed OSC2_FREQ_R_MAIN
- net OSC2_Freq_R_Ctrl renamed OSC2_FREQ_R_CTRL
- net OSC2_LFO_Cap renamed OSC2_LFO_CAP_MAIN
- net OSC2_LFO_Cap_Ctrl renamed OSC2_LFO_CAP_CTRL
- net OSC2_LFO_Main renamed OSC2_LFO_MAIN
- net OSC2_LFO_Main_Ctrl renamed OSC2_LFO_CTRL
- net OSC2_LFO_Signal renamed OSC2_FILTER_MOD_MAIN
- net OSC2_Signal renamed OSC2_SIGNAL_MAIN
- net OSC2_Signal_Ctrl renamed OSC2_SIGNAL_CTRL
- net PIEZO_NORMAL_MAIN: no longer names the net of J5.3 (Pin_3)
- net PIEZO_NORMAL_MAIN: no longer J4.2 (Pin_2)
- net Res_Amount renamed RES_AMOUNT_MAIN
- net Res_Amount_Ctrl renamed RES_AMOUNT_CTRL
- net Res_Top renamed RES_TOP_MAIN
- net Res_Top_Ctrl renamed RES_TOP_CTRL
- new net: C9.2, R14.1, U1.1, U1.2
- new net: D5.2 (A), R76.2
- no-connect marks 11 -> 10
Other:
- moved on the sheet: C1, C10, C11, C12, C13, C3, C6, C7, C9, D3, D4, D5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
