File: kicad/magnum-drum-synth.kicad_sch (KiCad schematic)
At the start: 125 parts, among them J10 Conn_01x04_Header, J11 Conn_01x04_Socket, J12 Eurorack Mono Jack, J18 Eurorack Mono Jack, J2 Eurorack Mono Jack, J26 Eurorack Mono Jack, J3 Conn_01x04_Socket, J4 Conn_01x04_Header, J5 Conn_01x03_Header, J6 Conn_01x06_Header, J7 Conn_01x06_Socket, J8 Conn_01x06_Header, J9 Conn_01x06_Socket, Q1 2N3904, Q2 2N3904, Q3 2N3904, Q4 2N3904, Q5 2N3904, Q6 2N3906, Q7 2N3906, Q8 2N3906, Q9 2N3906, SW1 DPDT, U1 CD4093, U3 TL074, U4 TL074, U7 LM13700

Commit message: Final fixes and tweaks (hopefully)
Parts:
- removed C5: 100nF, rumblesan-standard-parts:C_Rect_L7.0mm_W3.5mm_P5.00mm, symbol Device:C
- removed J10, J4: Conn_01x04_Header, Connector_PinHeader_2.54mm:PinHeader_1x04_P2.54mm_Vertical, symbol Connector:Conn_01x04_Male
- removed J11, J3: Conn_01x04_Socket, Connector_PinSocket_2.54mm:PinSocket_1x04_P2.54mm_Vertical, symbol Connector:Conn_01x04_Female
- removed J6, J8: Conn_01x06_Header, Connector_PinHeader_2.54mm:PinHeader_1x06_P2.54mm_Vertical, symbol Connector:Conn_01x06_Male
- removed J7, J9: Conn_01x06_Socket, Connector_PinSocket_2.54mm:PinSocket_1x06_P2.54mm_Vertical, symbol Connector:Conn_01x06_Female
- removed Q2, Q3: 2N3904, rumblesan-standard-parts:TO-92_Inline_Wide, symbol Transistor_BJT:2N3904
- removed Q9: 2N3906, rumblesan-standard-parts:TO-92_Inline_Wide, symbol Transistor_BJT:2N3906
- removed R7, R9: 10k, rumblesan-standard-parts:R_Axial_DIN0207_L6.3mm_D2.5mm_P10.16mm_Horizontal, symbol Device:R
- removed R73: 22k, rumblesan-standard-parts:R_Axial_DIN0207_L6.3mm_D2.5mm_P10.16mm_Horizontal, symbol Device:R
- removed R74: 82k, rumblesan-standard-parts:R_Axial_DIN0207_L6.3mm_D2.5mm_P10.16mm_Horizontal, symbol Device:R
- removed R8: 22r, rumblesan-standard-parts:R_Axial_DIN0207_L6.3mm_D2.5mm_P10.16mm_Horizontal, symbol Device:R
- removed unit 2 of U4
- added C5: 1uF, rumblesan-standard-parts:CP_Radial_D5.0mm_P2.00mm, symbol Device:C_Polarized
- added J1: Conn_02x10_Odd_Even, Connector_PinHeader_2.54mm:PinHeader_2x10_P2.54mm_Vertical, symbol Connector_Generic:Conn_02x10_Odd_Even
- added J3: Conn_02x10_Odd_Even, Connector_PinSocket_2.54mm:PinSocket_2x10_P2.54mm_Vertical, symbol Connector_Generic:Conn_02x10_Odd_Even
- added RV13: 1mB, rumblesan-standard-parts:Potentiometer_THT_Bourns_3306P_Vertical, symbol rumblesan-standard-parts:R_Potentiometer_Trim
- added U2: TL072, rumblesan-standard-parts:DIP-8_W7.62mm_Socket, symbol Amplifier_Operational:TL072
- added unit 1 of U4
- R4: value 1m -> 1k
- R5: value 100k -> 220k
- TP10: value Mixer TestPoint -> Filter Output TestPoint
- TP11: value Mixer TestPoint -> Final Output TestPoint
- TP7: value TestPoint -> Filter CV Mixer TestPoint
- TP8: value Filter Env TestPoint -> Filter Envelope TestPoint
- TP9: value TestPoint -> VCA Envelope TestPoint
Connections:
- net +12V: no longer R4.1
- net AMP_DECAY_CV_MIX_CTRL: now also J3.18 (Pin_18)
- net AMP_DECAY_CV_MIX_MAIN: now also J1.18 (Pin_18)
- net FILTER_ENV_DECAY_CTRL: now also J3.19 (Pin_19)
- net FILTER_ENV_DECAY_MAIN: now also J1.19 (Pin_19)
- net FILTER_ENV_MOD_CTRL: now also J3.16 (Pin_16)
- net FILTER_ENV_MOD_MAIN: now also J1.16 (Pin_16)
- net FILTER_FREQ_CV_CTRL: now also J3.20 (Pin_20)
- net FILTER_FREQ_CV_MAIN: now also J1.20 (Pin_20)
- net FINAL_OUTPUT_CTRL: now also J3.14 (Pin_14)
- net FINAL_OUTPUT_MAIN: now also J1.14 (Pin_14)
- net GND: now also R5.1, U2.5 (+); no longer R5.2
- net MIX_RETURN_CTRL: now also J3.17 (Pin_17)
- net MIX_RETURN_MAIN: now also J1.17 (Pin_17)
- net NOISE_SIGNAL_CTRL: now also J3.1 (Pin_1)
- net NOISE_SIGNAL_MAIN: now also J1.1 (Pin_1), RV13.2, RV13.3, U2.7
- net OSC1_FREQ_L_CTRL: now also J3.4 (Pin_4)
- net OSC1_FREQ_L_MAIN: now also J1.4 (Pin_4)
- net OSC1_FREQ_R_CTRL: now also J3.2 (Pin_2)
- net OSC1_FREQ_R_MAIN: now also U1.11, J1.2 (Pin_2); no longer U1.10
- net OSC1_SIGNAL_CTRL: now also J3.7 (Pin_7)
- net OSC1_SIGNAL_MAIN: now also J1.7 (Pin_7)
- net OSC2_FILTER_MOD_CTRL: now also J3.9 (Pin_9)
- net OSC2_FILTER_MOD_MAIN: now also J1.9 (Pin_9), U2.1, U2.2 (-)
- net OSC2_FREQ_L_CTRL: now also J3.6 (Pin_6)
- net OSC2_FREQ_L_MAIN: now also J1.6 (Pin_6)
- net OSC2_FREQ_R_CTRL: now also J3.8 (Pin_8)
- net OSC2_FREQ_R_MAIN: now also U1.10, J1.8 (Pin_8); no longer U1.11
- net OSC2_LFO_CAP_CTRL: now also J3.10 (Pin_10)
- net OSC2_LFO_CAP_MAIN: now also J1.10 (Pin_10)
- net OSC2_LFO_CTRL: now also J3.12 (Pin_12)
- net OSC2_LFO_MAIN: now also U1.8, U1.9, C5.1, J1.12 (Pin_12); no longer U1.12, U1.13
- net OSC2_SIGNAL_CTRL: now also J3.5 (Pin_5)
- net OSC2_SIGNAL_MAIN: now also J1.5 (Pin_5)
- net PIEZO_CTRL: now also J3.11 (Pin_11)
- net PIEZO_MAIN: now also J1.11 (Pin_11)
- net RES_AMOUNT_CTRL: now also J3.13 (Pin_13)
- net RES_AMOUNT_MAIN: now also J1.13 (Pin_13)
- net RES_TOP_CTRL: now also J3.15 (Pin_15)
- net RES_TOP_MAIN: now also J1.15 (Pin_15)
- net TRIG_IN_CTRL: now also J3.3 (Pin_3)
- net TRIG_IN_MAIN: now also J1.3 (Pin_3)
- net at C16.1, D6.1 (K), U7.5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: now also U4.3 (+)
- net at R42.1, TP9.1: now also U4.1, U4.2 (-)
- net at C2.2, R2.1: now also U1.12, U1.13; no longer U1.8, U1.9
- new net: C5.2, R5.2, U2.3 (+)
- new net: C4.2, R4.1
- new net: R4.2, RV13.1, U2.6 (-)
Other:
- moved on the sheet: C10, R15, R16, R17, R18, RV2, RV3, RV4, RV5, RV6, SW1A, SW1B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

Commit message: geographically reannotate all the parts
Parts:
- renumbered C12 to C1, C4 to C11, C2 to C12, C7 to C15, C3 to C16, C9 to C17, C5 to C18, C11 to C19, C10 to C2, C6 to C20, C13 to C23, C1 to C24, C16 to C29, C8 to C3, C15 to C36, C14 to C6, C36 to C7, D4 to D5, D3 to D6, D5 to D7, D6 to D8, H10 to H1, H8 to H10, H9 to H2, H7 to H9, J3 to J1, J18 to J10, J26 to J11, J5 to J4, J1 to J7, J2 to J8, J12 to J9, Q4 to Q2, Q6 to Q3, Q5 to Q4, Q7 to Q5, Q8 to Q6, R35 to R1, R24 to R10, R18 to R11, R25 to R12, R11 to R13, R27 to R14, R30 to R15, R33 to R16, R12 to R17, R6 to R18, R10 to R19, R15 to R2, R31 to R20, R1 to R21, R13 to R22, R2 to R23, R4 to R24, R14 to R25, R5 to R26, R75 to R27, R38 to R29, R17 to R3, R26 to R34, R76 to R35, R3 to R36, R16 to R4, R41 to R44, R37 to R45, R28 to R46, R23 to R5, R29 to R51, R42 to R59, R20 to R6, R32 to R60, R39 to R61, R36 to R63, R40 to R68, R22 to R7, R34 to R71, R19 to R8, R21 to R9, RV7 to RV10, RV8 to RV11, RV11 to RV12, RV10 to RV13, RV13 to RV2, RV5 to RV3, RV2 to RV4, RV6 to RV5, RV3 to RV6, RV4 to RV7, RV12 to RV8, TP12 to TP10, TP9 to TP11, TP10 to TP12, TP4 to TP2, TP5 to TP3, TP3 to TP4, TP2 to TP5, TP8 to TP6, TP11 to TP7, TP6 to TP8, TP7 to TP9, U3 to U1, U1 to U2, U2 to U3, U4 to U5, U7 to U6
