File: kicad/magnum-drum-synth.kicad_sch (KiCad schematic)
At the start: 113 parts, among them J1 Conn_02x10_Odd_Even, J10 Eurorack Mono Jack, J11 Eurorack Mono Jack, J4 Conn_01x03_Header, J7 Conn_02x10_Odd_Even, J8 Eurorack Mono Jack, J9 Eurorack Mono Jack, Q1 2N3904, Q2 2N3904, Q3 2N3906, Q4 2N3904, Q5 2N3906, Q6 2N3906, SW1 DPDT, U1 TL074, U2 CD4093, U3 TL072, U5 TL074, U6 LM13700

Commit message: Update kicad project for v7
Parts:
- C1, C11, C12, C16, C19, C2, C3, C6, C7: footprint rumblesan-standard-parts:C_Rect_L7.0mm_W3.5mm_P5.00mm -> Rumblesan_Standard_Parts:C_Rect_L7.0mm_W3.5mm_P5.00mm
- C15, C17, C18, C20, C23, C24, C36: footprint rumblesan-standard-parts:CP_Radial_D5.0mm_P2.00mm -> Rumblesan_Standard_Parts:CP_Radial_D5.0mm_P2.00mm
- C29: footprint rumblesan-standard-parts:C_Radial_D5.0mm_H5.0mm_P2.00mm -> Rumblesan_Standard_Parts:C_Radial_D5.0mm_H5.0mm_P2.00mm
- D1, D2, D5, D6, D7, D8: footprint rumblesan-standard-parts:D_DO-35_SOD27_P7.62mm_Horizontal -> Rumblesan_Standard_Parts:D_DO-35_SOD27_P7.62mm_Horizontal
- H1, H10, H2, H9: footprint rumblesan-standard-parts:MountingHole_3.2mm_M3_DIN965_Pad -> Rumblesan_Standard_Parts:MountingHole_3.2mm_M3_DIN965_Pad
- J10, J11, J8, J9: footprint rumblesan-standard-parts:Jack_3.5mm_QingPu_WQP-PJ398SM_Vertical -> Rumblesan_Standard_Parts:Jack_3.5mm_QingPu_WQP-PJ398SM_Vertical; symbol Eurorack_Hardware:Eurorack Mono Jack -> Audio_Connectors:Eurorack_Mono_Jack
- J4: symbol Connector:Conn_01x03_Male -> Connector:Conn_01x03_Pin
- MK1: symbol rumblesan-standard-parts:Piezo -> Rumblesan Standard Parts:Piezo
- Q1, Q2, Q3, Q4, Q5, Q6: footprint rumblesan-standard-parts:TO-92_Inline_Wide -> Rumblesan_Standard_Parts:TO-92_Inline_Wide
- R1, R10, R11, R12, R13, R14, R15, R16, R17, R18, R19, R2, R20, R21, R22, R23, R24, R25, R26, R27, R29, R3, R34, R35, R36, R4, R44, R45, R46, R5, R51, R59, R6, R60, R61, R63, R68, R7, R71, R8, R9: footprint rumblesan-standard-parts:R_Axial_DIN0207_L6.3mm_D2.5mm_P10.16mm_Horizontal -> Rumblesan_Standard_Parts:R_Axial_DIN0207_L6.3mm_D2.5mm_P10.16mm_Horizontal
- RV1: footprint rumblesan-standard-parts:Potentiometer_THT_Bourns_3306P_Vertical -> Rumblesan_Standard_Parts:Potentiometer_THT_Bourns_3306P_Vertical
- RV10, RV11, RV12, RV13, RV8, RV9: footprint rumblesan-standard-parts:Potentiometer_Alpha_RD901F-40-00D_Single_Vertical_CircularHoles -> Rumblesan_Standard_Parts:Potentiometer_Alpha_RD901F-40-00D_Single_Vertical_CircularHoles
- RV2: footprint rumblesan-standard-parts:Potentiometer_THT_Bourns_3306P_Vertical -> Rumblesan_Standard_Parts:Potentiometer_THT_Bourns_3306P_Vertical; symbol rumblesan-standard-parts:R_Potentiometer_Trim -> Rumblesan Standard Parts:R_Potentiometer_Trim
- RV3, RV4, RV5, RV6, RV7: footprint rumblesan-standard-parts:Potentiometer_Song_Huei_R0904N_Single_Vertical -> Rumblesan_Standard_Parts:Potentiometer_Song_Huei_R0904N_Single_Vertical
- SW1: footprint rumblesan-standard-parts:SW_PUSH_2P2T_8mm_Apem_MHPS2285 -> Rumblesan_Standard_Parts:SW_PUSH_2P2T_8mm_Apem_MHPS2285
- TP1, TP10, TP11, TP12, TP2, TP3, TP4, TP5, TP6, TP7, TP8, TP9: footprint rumblesan-standard-parts:TestPoint_Loop_D2.50mm_Drill1.0mm_LowProfile -> Rumblesan_Standard_Parts:TestPoint_Loop_D2.50mm_Drill1.0mm_LowProfile
- U1, U2, U5: footprint rumblesan-standard-parts:DIP-14_W7.62mm_Socket -> Rumblesan_Standard_Parts:DIP-14_W7.62mm_Socket
- U3: footprint rumblesan-standard-parts:DIP-8_W7.62mm_Socket -> Rumblesan_Standard_Parts:DIP-8_W7.62mm_Socket
- U6: footprint rumblesan-standard-parts:DIP-16_W7.62mm_Socket -> Rumblesan_Standard_Parts:DIP-16_W7.62mm_Socket
Connections:
- net FINAL_OUTPUT_CTRL: now also J11.2 (Tip); no longer J11.T (Tip)
- net GND: now also J10.1 (Sleeve), J11.1 (Sleeve), J8.1 (Sleeve), J9.1 (Sleeve); no longer J10.S (Sleeve), J11.S (Sleeve), J8.S (Sleeve), J9.S (Sleeve)
- net PIEZO_CTRL: now also J8.3 (Tip_normalize); no longer J8.TN (Tip_normalize)
- net TRIG_IN_CTRL: now also J8.2 (Tip); no longer J8.T (Tip)
- net at R6.1: now also J9.2 (Tip); no longer J9.T (Tip)
- net at R15.1: now also J10.2 (Tip); no longer J10.T (Tip)

Commit message: Final board tweaks
Parts:
- removed C11: 100nF, Rumblesan_Standard_Parts:C_Rect_L7.0mm_W3.5mm_P5.00mm, symbol Device:C
- removed Q1: 2N3904, Rumblesan_Standard_Parts:TO-92_Inline_Wide, symbol Transistor_BJT:2N3904
- added C1, C2: 100nF, Rumblesan_Standard_Parts:C_Rect_L7.0mm_W3.5mm_P5.00mm, symbol Rumblesan Standard Parts:C
- added C37: 100nF, Rumblesan_Standard_Parts:C_Rect_L7.0mm_W3.5mm_P5.00mm, symbol Device:C
- added Q1: 293904, Rumblesan_Standard_Parts:TO-92_Inline_Wide, symbol Transistor_BJT:BC547
- added Q2: 2n3904, Rumblesan_Standard_Parts:TO-92_Inline_Wide, symbol Transistor_BJT:2N3904
- added R12: 10k, Rumblesan_Standard_Parts:R_Axial_DIN0207_L6.3mm_D2.5mm_P10.16mm_Horizontal, symbol Rumblesan Standard Parts:R
- added R3: 560k, Rumblesan_Standard_Parts:R_Axial_DIN0207_L6.3mm_D2.5mm_P10.16mm_Horizontal, symbol Rumblesan Standard Parts:R
- added R4: 22r, Rumblesan_Standard_Parts:R_Axial_DIN0207_L6.3mm_D2.5mm_P10.16mm_Horizontal, symbol Rumblesan Standard Parts:R
- added R6: 100k, Rumblesan_Standard_Parts:R_Axial_DIN0207_L6.3mm_D2.5mm_P10.16mm_Horizontal, symbol Rumblesan Standard Parts:R
- R2: value 4k7 -> 100k
- R24: value 1k -> 10k
- R25: value 150k -> 100k
- R29: value 470r -> 100r
- R44: value 1k -> 470r
- R46: value 47r -> 10k
- R51: value 470r -> 1k
- R59: value 47k -> 18k
- R68: value 100k -> 33k
- RV2: value 1mB -> 1m
Connections:
- net +12V: now also R12.2, R3.2
- net FILTER_FREQ_CV_MAIN: now also Q4.2 (B), R51.1; no longer R46.1
- net GND: now also R27.1, R46.2, Q1.2 (B), R4.1, R6.1
- net MIX_RETURN_CTRL: now also J1.13 (Pin_13); no longer J1.17 (Pin_17)
- net MIX_RETURN_MAIN: now also J7.13 (Pin_13); no longer J7.17 (Pin_17)
- net OSC2_FILTER_MOD_CTRL: now also J1.11 (Pin_11); no longer J1.9 (Pin_9)
- net OSC2_FILTER_MOD_MAIN: now also J7.11 (Pin_11); no longer J7.9 (Pin_9)
- net OSC2_FREQ_L_CTRL: now also J1.8 (Pin_8); no longer J1.6 (Pin_6)
- net OSC2_FREQ_L_MAIN: now also J7.8 (Pin_8); no longer J7.6 (Pin_6)
- net OSC2_FREQ_R_CTRL: now also J1.6 (Pin_6); no longer J1.8 (Pin_8)
- net OSC2_FREQ_R_MAIN: now also J7.6 (Pin_6); no longer J7.8 (Pin_8)
- net OSC2_LFO_CAP_CTRL: now also J1.12 (Pin_12), SW1.2 (B); no longer J1.10 (Pin_10), SW1.1 (A)
- net OSC2_LFO_CAP_MAIN: now also J7.12 (Pin_12); no longer J7.10 (Pin_10)
- net OSC2_LFO_CTRL: now also J1.10 (Pin_10), SW1.1 (A); no longer J1.12 (Pin_12), SW1.2 (B)
- net OSC2_LFO_MAIN: now also J7.10 (Pin_10); no longer J7.12 (Pin_12)
- net OSC2_SIGNAL_CTRL: now also J1.9 (Pin_9); no longer J1.5 (Pin_5)
- net OSC2_SIGNAL_MAIN: now also J7.9 (Pin_9); no longer J7.5 (Pin_5)
- net PIEZO_CTRL: now also J1.5 (Pin_5); no longer J1.11 (Pin_11)
- net PIEZO_MAIN: now also J4.3 (Pin_3), J7.5 (Pin_5); no longer J4.2 (Pin_2), J7.11 (Pin_11)
- net RES_AMOUNT_CTRL: now also J1.15 (Pin_15); no longer J1.13 (Pin_13)
- net RES_AMOUNT_MAIN: now also J7.15 (Pin_15); no longer J7.13 (Pin_13)
- net RES_TOP_CTRL: now also J1.17 (Pin_17); no longer J1.15 (Pin_15)
- net RES_TOP_MAIN: now also J7.17 (Pin_17); no longer J7.15 (Pin_15)
- net at R21.2: now also C1.1, Q1.3 (E)
- net at D5.1 (K), D6.1 (K), TP2.1: now also R27.2, C37.2; no longer R27.1
- net at D6.2 (A): now also J4.2 (Pin_2); no longer J4.1 (Pin_1)
- net at R24.1: now also C2.2
- net at C19.2, Q2.2 (B): now also R46.1, C37.1; no longer R27.2
- new net: C2.1, Q2.3 (C), R12.1
- new net: C1.2, Q2.2 (B), R3.1, R6.2
- new net: Q2.1 (E), R4.2
Other:
- note added: "should see roughly 8V peak"
- moved on the sheet: C17, C19, Q2, R22, R24, R25, R27, RV2, TP1, TP3, U2A, U2B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

Commit message: Final tweaks
Parts:
- removed Q1: 293904, Rumblesan_Standard_Parts:TO-92_Inline_Wide, symbol Transistor_BJT:BC547
- added H13, H14, H15, H16: MountingHole_Pad, Rumblesan_Standard_Parts:MountingHole_3.2mm_M3_DIN965_Pad, symbol Mechanical:MountingHole_Pad
- added Q7: 2N3904, Rumblesan_Standard_Parts:TO-92_Inline_Wide, symbol Transistor_BJT:2N3904
- Q2: value 2n3904 -> 2N3904
- R25: value 100k -> 10k
- SW1: PartNumber MHPS2285 -> (none); mpn (none) -> MHPS2285
Connections:
- net GND: now also H13.1, H14.1, H15.1, H16.1, Q7.2 (B)
- net at C1.1, R21.2: now also Q7.1 (E)
Other:
- note added: "envelope should be roughly 10V peak"
- note added: "range should be 3.1v to 450mV"
- note added: "trigger should be 12v and 8ms wide"
- note removed: "should see roughly 8V peak"
