File: kicad/filter.kicad_sch (KiCad schematic)
At the start: 31 parts, among them U5 LM13700, U6 LM13700

Commit message: geographically reannotate all the parts
Parts:
- renumbered C17 to C21, C19 to C27, C18 to C30, C20 to C33, R44 to R28, R56 to R30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
