File: kicad/filter.kicad_sch (KiCad schematic)
At the start: 31 parts, among them U4 LM13700, U7 LM13700

Commit message: Update kicad project for v7
Parts:
- C21, C27, C30, C33: footprint rumblesan-standard-parts:C_Rect_L7.0mm_W3.5mm_P5.00mm -> Rumblesan_Standard_Parts:C_Rect_L7.0mm_W3.5mm_P5.00mm
- R28, R30, R31, R32, R33, R37, R38, R39, R40, R41, R42, R43, R47, R48, R52, R53, R54, R55, R56, R57, R58, R64, R65, R66, R70: footprint rumblesan-standard-parts:R_Axial_DIN0207_L6.3mm_D2.5mm_P10.16mm_Horizontal -> Rumblesan_Standard_Parts:R_Axial_DIN0207_L6.3mm_D2.5mm_P10.16mm_Horizontal
- U4, U7: footprint rumblesan-standard-parts:DIP-16_W7.62mm_Socket -> Rumblesan_Standard_Parts:DIP-16_W7.62mm_Socket
