File: kicad/output-vca.kicad_sch (KiCad schematic)
At the start: 8 parts, among them J27 Conn_01x03_Header, U2 TL072, U7 LM13700

Commit message: Tweaking schematic and bom values
Parts:
- R71: value 33k -> 68k
- R72: value 10k -> 33k
Changed lines of the file:
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@@
   (symbol (lib_id "Device:R") (at 154.94 67.31 90) (unit 1)
     (in_bom yes) (on_board yes) (fields_autoplaced)
-    (property "Reference" "R71" (id 0) (at 154.94 62.3275 90))
-    (property "Value" "33k" (id 1) (at 154.94 65.1026 90))
+    (property "Reference" "R71" (id 0) (at 154.94 62.5942 90))
+    (property "Value" "68k" (id 1) (at 154.94 65.1311 90))
     (property "Footprint" "rumblesan-standard-parts:R_Axial_DIN0207_L6.3mm_D2.5mm_P10.16mm_Horizontal" (id 2) (at 154.94 69.088 90)
       (effects (font (size 1.27 1.27)) hide)
@@
     (in_bom yes) (on_board yes)
     (property "Reference" "R72" (id 0) (at 154.94 74.93 90))
-    (property "Value" "10k" (id 1) (at 154.94 70.1826 90))
+    (property "Value" "33k" (id 1) (at 154.94 70.1826 90))
     (property "Footprint" "rumblesan-standard-parts:R_Axial_DIN0207_L6.3mm_D2.5mm_P10.16mm_Horizontal" (id 2) (at 154.94 74.168 90)
       (effects (font (size 1.27 1.27)) hide)

Commit message: Final tweaks to rev 4
Parts:
- R71: value 68k -> 100k
Changed lines of the file:
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@@
   (title_block
     (title "Magnum Percussion Instrument")
-    (date "2022-06-15")
-    (rev "r03")
+    (date "2022-09-29")
+    (rev "r04")
     (comment 2 "creativecommons.org/licenses/by/4.0/")
     (comment 3 "License: CC BY 4.0")
@@
     (in_bom yes) (on_board yes) (fields_autoplaced)
     (property "Reference" "R71" (id 0) (at 154.94 62.5942 90))
-    (property "Value" "68k" (id 1) (at 154.94 65.1311 90))
+    (property "Value" "100k" (id 1) (at 154.94 65.1311 90))
     (property "Footprint" "rumblesan-standard-parts:R_Axial_DIN0207_L6.3mm_D2.5mm_P10.16mm_Horizontal" (id 2) (at 154.94 69.088 90)
       (effects (font (size 1.27 1.27)) hide)

Commit message: slimlining opamp count and more moving around
Parts:
- removed U2: TL072, rumblesan-standard-parts:DIP-8_W7.62mm_Socket, symbol Amplifier_Operational:TL072
- added U4: TL074, rumblesan-standard-parts:DIP-14_W7.62mm_Socket, symbol Amplifier_Operational:TL074
Connections:
- net GND: now also U4.3 (+)
- net Output: now also U4.1
- net at J27.2 (Pin_2), U7.12: now also U4.2 (-)
Changed lines of the file:
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@@
     (pin "2")
+  )
+  (symbol (lib_id "Amplifier_Operational:TL074") (at 157.48 88.9 0) (mirror x) (unit 1)
+    (in_bom yes) (on_board yes) (fields_autoplaced)
+    (property "Reference" "U4" (id 0) (at 157.48 79.8535 0))
+    (property "Value" "TL074" (id 1) (at 157.48 82.6286 0))
+    (property "Footprint" "rumblesan-standard-parts:DIP-14_W7.62mm_Socket" (id 2) (at 156.21 91.44 0)
+      (effects (font (size 1.27 1.27)) hide)
+    )
+    (property "Datasheet" "http://www.ti.com/lit/ds/symlink/tl071.pdf" (id 3) (at 158.75 93.98 0)
+      (effects (font (size 1.27 1.27)) hide)
+    )
+    (pin "1")
+    (pin "2")
+    (pin "3")
+    (pin "5")
+    (pin "6")
+    (pin "7")
+    (pin "10")
+    (pin "8")
+    (pin "9")
+    (pin "12")
+    (pin "13")
+    (pin "14")
+    (pin "11")
+    (pin "4")
   )
   (symbol (lib_id "Amplifier_Operational:LM13700") (at 127 86.36 0) (unit 1)
@@
     (pin "2")
   )
-  (symbol (lib_id "Amplifier_Operational:TL072") (at 157.48 88.9 0) (mirror x) (unit 1)
-    (in_bom yes) (on_board yes) (fields_autoplaced)
-    (property "Reference" "U2" (id 0) (at 157.48 79.8535 0))
-    (property "Value" "TL072" (id 1) (at 157.48 82.6286 0))
-    (property "Footprint" "rumblesan-standard-parts:DIP-8_W7.62mm_Socket" (id 2) (at 157.48 88.9 0)
-      (effects (font (size 1.27 1.27)) hide)
-    )
-    (property "Datasheet" "http://www.ti.com/lit/ds/symlink/tl071.pdf" (id 3) (at 157.48 88.9 0)
-      (effects (font (size 1.27 1.27)) hide)
-    )
-    (pin "1")
-    (pin "2")
-    (pin "3")
-    (pin "5")
-    (pin "6")
-    (pin "7")
-    (pin "4")
-    (pin "8")
-  )
   (symbol (lib_id "power:GND") (at 115.57 102.87 0) (unit 1)

Commit message: Final fixes and tweaks (hopefully)
Parts:
- removed U4: TL074, rumblesan-standard-parts:DIP-14_W7.62mm_Socket, symbol Amplifier_Operational:TL074
- added U4: TL074, rumblesan-standard-parts:DIP-14_W7.62mm_Socket, symbol Amplifier_Operational:TL074
Connections:
- net GND: now also U4.5 (+)
- net Output: now also U4.7
- net at J27.2 (Pin_2), U7.12: now also U4.6 (-)
Changed lines of the file:
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@@
     (pin "2")
   )
-  (symbol (lib_id "Amplifier_Operational:TL074") (at 157.48 88.9 0) (mirror x) (unit 1)
+  (symbol (lib_id "Connector:Conn_01x03_Male") (at 140.97 69.85 0) (unit 1)
+    (in_bom yes) (on_board yes)
+    (property "Reference" "J27" (id 0) (at 140.97 74.93 0))
+    (property "Value" "Conn_01x03_Header" (id 1) (at 141.605 66.0424 0)
+      (effects (font (size 1.27 1.27)) hide)
+    )
+    (property "Footprint" "Connector_PinHeader_2.54mm:PinHeader_1x03_P2.54mm_Vertical" (id 2) (at 140.97 69.85 0)
+      (effects (font (size 1.27 1.27)) hide)
+    )
+    (property "Datasheet" "~" (id 3) (at 140.97 69.85 0)
+      (effects (font (size 1.27 1.27)) hide)
+    )
+    (property "Name" "Output Level Select" (id 4) (at 140.97 63.5 0))
+    (pin "1")
+    (pin "2")
+    (pin "3")
+  )
+  (symbol (lib_id "Device:R") (at 154.94 72.39 90) (unit 1)
+    (in_bom yes) (on_board yes)
+    (property "Reference" "R72" (id 0) (at 154.94 74.93 90))
+    (property "Value" "33k" (id 1) (at 154.94 70.1826 90))
+    (property "Footprint" "rumblesan-standard-parts:R_Axial_DIN0207_L6.3mm_D2.5mm_P10.16mm_Horizontal" (id 2) (at 154.94 74.168 90)
+      (effects (font (size 1.27 1.27)) hide)
+    )
+    (property "Datasheet" "~" (id 3) (at 154.94 72.39 0)
+      (effects (font (size 1.27 1.27)) hide)
+    )
+    (property "Tolerance" "1%" (id 4) (at 154.94 72.39 0)
+      (effects (font (size 1.27 1.27)) hide)
+    )
+    (pin "1")
+    (pin "2")
+  )
+  (symbol (lib_id "Amplifier_Operational:TL074") (at 157.48 88.9 0) (mirror x) (unit 2)
     (in_bom yes) (on_board yes) (fields_autoplaced)
     (property "Reference" "U4" (id 0) (at 157.48 79.8535 0))
@@
     (pin "6")
   )
-  (symbol (lib_id "Connector:Conn_01x03_Male") (at 140.97 69.85 0) (unit 1)
-    (in_bom yes) (on_board yes)
-    (property "Reference" "J27" (id 0) (at 140.97 74.93 0))
-    (property "Value" "Conn_01x03_Header" (id 1) (at 141.605 66.0424 0)
-      (effects (font (size 1.27 1.27)) hide)
-    )
-    (property "Footprint" "Connector_PinHeader_2.54mm:PinHeader_1x03_P2.54mm_Vertical" (id 2) (at 140.97 69.85 0)
-      (effects (font (size 1.27 1.27)) hide)
-    )
-    (property "Datasheet" "~" (id 3) (at 140.97 69.85 0)
-      (effects (font (size 1.27 1.27)) hide)
-    )
-    (property "Name" "Output Level Select" (id 4) (at 140.97 63.5 0))
-    (pin "1")
-    (pin "2")
-    (pin "3")
-  )
-  (symbol (lib_id "Device:R") (at 154.94 72.39 90) (unit 1)
-    (in_bom yes) (on_board yes)
-    (property "Reference" "R72" (id 0) (at 154.94 74.93 90))
-    (property "Value" "33k" (id 1) (at 154.94 70.1826 90))
-    (property "Footprint" "rumblesan-standard-parts:R_Axial_DIN0207_L6.3mm_D2.5mm_P10.16mm_Horizontal" (id 2) (at 154.94 74.168 90)
-      (effects (font (size 1.27 1.27)) hide)
-    )
-    (property "Datasheet" "~" (id 3) (at 154.94 72.39 0)
-      (effects (font (size 1.27 1.27)) hide)
-    )
-    (property "Tolerance" "1%" (id 4) (at 154.94 72.39 0)
-      (effects (font (size 1.27 1.27)) hide)
-    )
-    (pin "1")
-    (pin "2")
-  )
   (symbol (lib_id "power:GND") (at 115.57 102.87 0) (unit 1)
     (in_bom yes) (on_board yes) (fields_autoplaced)
@@
     (pin "1")
     (pin "2")
+  )
+  (symbol (lib_id "Amplifier_Operational:LM13700") (at 185.42 57.15 0) (unit 2)
+    (in_bom yes) (on_board yes) (fields_autoplaced)
+    (property "Reference" "U7" (id 0) (at 182.88 48.2399 0))
+    (property "Value" "LM13700" (id 1) (at 182.88 51.015 0))
+    (property "Footprint" "rumblesan-standard-parts:DIP-16_W7.62mm_Socket" (id 2) (at 177.8 56.515 0)
+      (effects (font (size 1.27 1.27)) hide)
+    )
+    (property "Datasheet" "http://www.ti.com/lit/ds/symlink/lm13700.pdf" (id 3) (at 177.8 56.515 0)
+      (effects (font (size 1.27 1.27)) hide)
+    )
+    (pin "12")
+    (pin "13")
+    (pin "14")
+    (pin "15")
+    (pin "16")
+    (pin "10")
+    (pin "9")
+    (pin "1")
+    (pin "2")
+    (pin "3")
+    (pin "4")
+    (pin "5")
+    (pin "7")
+    (pin "8")
+    (pin "11")
+    (pin "6")
   )
   (symbol (lib_id "Device:R") (at 106.68 96.52 0) (unit 1)
@@
     (pin "2")
   )
-  (symbol (lib_id "Amplifier_Operational:LM13700") (at 185.42 57.15 0) (unit 2)
-    (in_bom yes) (on_board yes) (fields_autoplaced)
-    (property "Reference" "U7" (id 0) (at 182.88 48.2399 0))
-    (property "Value" "LM13700" (id 1) (at 182.88 51.015 0))
-    (property "Footprint" "rumblesan-standard-parts:DIP-16_W7.62mm_Socket" (id 2) (at 177.8 56.515 0)
-      (effects (font (size 1.27 1.27)) hide)
-    )
-    (property "Datasheet" "http://www.ti.com/lit/ds/symlink/lm13700.pdf" (id 3) (at 177.8 56.515 0)
-      (effects (font (size 1.27 1.27)) hide)
-    )
-    (pin "12")
-    (pin "13")
-    (pin "14")
-    (pin "15")
-    (pin "16")
-    (pin "10")
-    (pin "9")
-    (pin "1")
-    (pin "2")
-    (pin "3")
-    (pin "4")
-    (pin "5")
-    (pin "7")
-    (pin "8")
-    (pin "11")
-    (pin "6")
-  )
   (symbol (lib_id "power:GND") (at 106.68 102.87 0) (unit 1)

Commit message: geographically reannotate all the parts
Parts:
- renumbered J27 to J5, R71 to R49, R72 to R50, R70 to R62, R69 to R67, R68 to R69, U4 to U5, U7 to U6
Changed lines of the file:
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@@
   (symbol (lib_id "Device:R") (at 154.94 67.31 90) (unit 1)
     (in_bom yes) (on_board yes) (fields_autoplaced)
-    (property "Reference" "R71" (id 0) (at 154.94 62.5942 90))
+    (property "Reference" "R49" (id 0) (at 154.94 62.5942 90))
     (property "Value" "100k" (id 1) (at 154.94 65.1311 90))
     (property "Footprint" "rumblesan-standard-parts:R_Axial_DIN0207_L6.3mm_D2.5mm_P10.16mm_Horizontal" (id 2) (at 154.94 69.088 90)
@@
   (symbol (lib_id "Connector:Conn_01x03_Male") (at 140.97 69.85 0) (unit 1)
     (in_bom yes) (on_board yes)
-    (property "Reference" "J27" (id 0) (at 140.97 74.93 0))
+    (property "Reference" "J5" (id 0) (at 140.97 74.93 0))
     (property "Value" "Conn_01x03_Header" (id 1) (at 141.605 66.0424 0)
       (effects (font (size 1.27 1.27)) hide)
@@
   (symbol (lib_id "Device:R") (at 154.94 72.39 90) (unit 1)
     (in_bom yes) (on_board yes)
-    (property "Reference" "R72" (id 0) (at 154.94 74.93 90))
+    (property "Reference" "R50" (id 0) (at 154.94 74.93 90))
     (property "Value" "33k" (id 1) (at 154.94 70.1826 90))
     (property "Footprint" "rumblesan-standard-parts:R_Axial_DIN0207_L6.3mm_D2.5mm_P10.16mm_Horizontal" (id 2) (at 154.94 74.168 90)
@@
   (symbol (lib_id "Amplifier_Operational:TL074") (at 157.48 88.9 0) (mirror x) (unit 2)
     (in_bom yes) (on_board yes) (fields_autoplaced)
-    (property "Reference" "U4" (id 0) (at 157.48 79.8535 0))
+    (property "Reference" "U5" (id 0) (at 157.48 79.8535 0))
     (property "Value" "TL074" (id 1) (at 157.48 82.6286 0))
     (property "Footprint" "rumblesan-standard-parts:DIP-14_W7.62mm_Socket" (id 2) (at 156.21 91.44 0)
@@
   (symbol (lib_id "Amplifier_Operational:LM13700") (at 127 86.36 0) (unit 1)
     (in_bom yes) (on_board yes) (fields_autoplaced)
-    (property "Reference" "U7" (id 0) (at 127 77.3135 0))
+    (property "Reference" "U6" (id 0) (at 127 77.3135 0))
     (property "Value" "LM13700" (id 1) (at 127 80.0886 0))
     (property "Footprint" "rumblesan-standard-parts:DIP-16_W7.62mm_Socket" (id 2) (at 119.38 85.725 0)
@@
   (symbol (lib_id "Device:R") (at 99.06 83.82 90) (unit 1)
     (in_bom yes) (on_board yes) (fields_autoplaced)
-    (property "Reference" "R68" (id 0) (at 99.06 78.8375 90))
+    (property "Reference" "R69" (id 0) (at 99.06 78.8375 90))
     (property "Value" "100k" (id 1) (at 99.06 81.6126 90))
     (property "Footprint" "rumblesan-standard-parts:R_Axial_DIN0207_L6.3mm_D2.5mm_P10.16mm_Horizontal" (id 2) (at 99.06 85.598 90)
@@
   (symbol (lib_id "Amplifier_Operational:LM13700") (at 185.42 57.15 0) (unit 2)
     (in_bom yes) (on_board yes) (fields_autoplaced)
-    (property "Reference" "U7" (id 0) (at 182.88 48.2399 0))
+    (property "Reference" "U6" (id 0) (at 182.88 48.2399 0))
     (property "Value" "LM13700" (id 1) (at 182.88 51.015 0))
     (property "Footprint" "rumblesan-standard-parts:DIP-16_W7.62mm_Socket" (id 2) (at 177.8 56.515 0)
@@
   (symbol (lib_id "Device:R") (at 106.68 96.52 0) (unit 1)
     (in_bom yes) (on_board yes) (fields_autoplaced)
-    (property "Reference" "R69" (id 0) (at 108.458 95.6115 0)
+    (property "Reference" "R67" (id 0) (at 108.458 95.6115 0)
       (effects (font (size 1.27 1.27)) (justify left))
     )
@@
   (symbol (lib_id "Device:R") (at 115.57 96.52 0) (unit 1)
     (in_bom yes) (on_board yes) (fields_autoplaced)
-    (property "Reference" "R70" (id 0) (at 117.348 95.6115 0)
+    (property "Reference" "R62" (id 0) (at 117.348 95.6115 0)
       (effects (font (size 1.27 1.27)) (justify left))
     )
