File: kicad/output-vca.kicad_sch (KiCad schematic)
At the start: 8 parts, among them J5 Conn_01x03_Header, U5 TL074, U6 LM13700

Commit message: Update kicad project for v7
Parts:
- J5: symbol Connector:Conn_01x03_Male -> Connector:Conn_01x03_Pin
- R49, R50, R62, R67, R69: footprint rumblesan-standard-parts:R_Axial_DIN0207_L6.3mm_D2.5mm_P10.16mm_Horizontal -> Rumblesan_Standard_Parts:R_Axial_DIN0207_L6.3mm_D2.5mm_P10.16mm_Horizontal
- U5: footprint rumblesan-standard-parts:DIP-14_W7.62mm_Socket -> Rumblesan_Standard_Parts:DIP-14_W7.62mm_Socket
- U6: footprint rumblesan-standard-parts:DIP-16_W7.62mm_Socket -> Rumblesan_Standard_Parts:DIP-16_W7.62mm_Socket

Commit message: Final board tweaks
Parts:
- R49: value 100k -> 56k
- R50: value 33k -> 12k
Changed lines of the file:
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@@
   (symbol (lib_id "Device:R") (at 154.94 67.31 90) (unit 1)
     (in_bom yes) (on_board yes) (dnp no) (fields_autoplaced)
-    (property "Reference" "R49" (at 154.94 62.5942 90)
+    (property "Reference" "R49" (at 154.94 62.23 90)
       (effects (font (size 1.27 1.27)))
     )
-    (property "Value" "100k" (at 154.94 65.1311 90)
+    (property "Value" "56k" (at 154.94 64.77 90)
       (effects (font (size 1.27 1.27)))
     )
@@
       (effects (font (size 1.27 1.27)))
     )
-    (property "Value" "33k" (at 154.94 70.1826 90)
+    (property "Value" "12k" (at 154.94 70.1826 90)
       (effects (font (size 1.27 1.27)))
     )
