File: kicad/magnum-drum-synth.kicad_pcb (KiCad board)
At the start: 2 copper layers, 202 x 105 mm, 179 parts, among them J1 Conn_02x10_Odd_Even, J10 Eurorack Mono Jack, J11 Eurorack Mono Jack, J2 Conn_01x04_Socket, J3 locked, J4 Conn_01x03_Header, J5 Conn_01x03_Header, J6 Conn_01x04_Header, J7 Conn_02x10_Odd_Even, J8 Eurorack Mono Jack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

Commit message: Final board tweaks
Parts:
- removed C11: 100nF, Rumblesan_Standard_Parts:C_Rect_L7.0mm_W3.5mm_P5.00mm
- removed Q1: 2N3904, Rumblesan_Standard_Parts:TO-92_Inline_Wide
- added C37: 100nF, Rumblesan_Standard_Parts:C_Rect_L7.0mm_W3.5mm_P5.00mm, F.Cu at (177.4, 59.6)
- added C38: 100nF, Rumblesan_Standard_Parts:C_Rect_L7.0mm_W3.5mm_P5.00mm, F.Cu at (223.0, 49.5)
- added C39: 100nF, Rumblesan_Standard_Parts:C_Rect_L7.0mm_W3.5mm_P5.00mm, F.Cu at (220.0, 40.1)
- added Q7: BC547, Rumblesan_Standard_Parts:TO-92_Inline_Wide, F.Cu at (214.6, 54.6)
- added Q8: BC549C, Rumblesan_Standard_Parts:TO-92_Inline_Wide, F.Cu at (227.6, 40.4)
- added R72: 560k, Rumblesan_Standard_Parts:R_Axial_DIN0207_L6.3mm_D2.5mm_P10.16mm_Horizontal, F.Cu at (219.7, 46.7)
- added R73: 100k, Rumblesan_Standard_Parts:R_Axial_DIN0207_L6.3mm_D2.5mm_P10.16mm_Horizontal, F.Cu at (226.6, 54.6)
- added R74: 10k, Rumblesan_Standard_Parts:R_Axial_DIN0207_L6.3mm_D2.5mm_P10.16mm_Horizontal, F.Cu at (219.7, 43.7)
- added R75: 22r, Rumblesan_Standard_Parts:R_Axial_DIN0207_L6.3mm_D2.5mm_P10.16mm_Horizontal, F.Cu at (229.6, 54.6)
- R2: value 4k7 -> 10k
- R24: value 1k -> 10k
- R25: value 150k -> 100k
- R29: value 470r -> 100r
- R44: value 1k -> 470r
- R46: value 47r -> 10k
- R49: value 100k -> 56k
- R50: value 33k -> 12k
- R51: value 470r -> 1k
- R59: value 47k -> 18k
- R68: value 100k -> 33k
- RV2: value 1mB -> 1m
- moved REF**2 64.2 mm to (161.0, 72.4)
- moved R46 40.2 mm to (155.1, 63.5), turned to 0 degrees
- moved R23 29.9 mm to (168.0, 66.2)
- moved R37 21.8 mm to (211.6, 61.5), turned to -90 degrees
- moved D4 20.4 mm to (146.4, 38.7), turned to -90 degrees
- moved TP1 17.2 mm to (187.7, 40.1)
- moved R21 16.6 mm to (209.6, 49.8)
- moved R25 15.7 mm to (160.9, 36.2)
- moved C23 13.1 mm to (167.0, 81.2)
- moved R36 12.8 mm to (168.0, 69.2), turned to 0 degrees
- moved R24 10.0 mm to (224.8, 36.6)
- moved R27 7.04 mm to (197.7, 55.5)
- moved Q2 6.99 mm to (162.7, 56.4), turned to 90 degrees
- moved TP6 6.56 mm to (177.3, 81.7)
- moved J4 6.31 mm to (193.2, 68.7), turned to -90 degrees
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Connections:
- J1 pad 10: /OSC2_LFO_CAP_CTRL -> /OSC2_LFO_CTRL
- J1 pad 11: /PIEZO_CTRL -> /OSC2_FILTER_MOD_CTRL
- J1 pad 12: /OSC2_LFO_CTRL -> /OSC2_LFO_CAP_CTRL
- J1 pad 13: /RES_AMOUNT_CTRL -> /MIX_RETURN_CTRL
- J1 pad 15: /RES_TOP_CTRL -> /RES_AMOUNT_CTRL
- J1 pad 17: /MIX_RETURN_CTRL -> /RES_TOP_CTRL
- J1 pad 5: /OSC2_SIGNAL_CTRL -> /PIEZO_CTRL
- J1 pad 6: /OSC2_FREQ_L_CTRL -> /OSC2_FREQ_R_CTRL
- J1 pad 8: /OSC2_FREQ_R_CTRL -> /OSC2_FREQ_L_CTRL
- J1 pad 9: /OSC2_FILTER_MOD_CTRL -> /OSC2_SIGNAL_CTRL
- J4 pad 1: Net-(D6-A) -> unconnected-(J4-Pin_1-Pad1)
- J4 pad 2: /PIEZO_MAIN -> Net-(D6-A)
- J4 pad 3: unconnected-(J4-Pin_3-Pad3) -> /PIEZO_MAIN
- J7 pad 10: /OSC2_LFO_CAP_MAIN -> /OSC2_LFO_MAIN
- J7 pad 11: /PIEZO_MAIN -> /OSC2_FILTER_MOD_MAIN
- J7 pad 12: /OSC2_LFO_MAIN -> /OSC2_LFO_CAP_MAIN
- J7 pad 13: /RES_AMOUNT_MAIN -> /MIX_RETURN_MAIN
- J7 pad 15: /RES_TOP_MAIN -> /RES_AMOUNT_MAIN
- J7 pad 17: /MIX_RETURN_MAIN -> /RES_TOP_MAIN
- J7 pad 5: /OSC2_SIGNAL_MAIN -> /PIEZO_MAIN
- J7 pad 6: /OSC2_FREQ_L_MAIN -> /OSC2_FREQ_R_MAIN
- J7 pad 8: /OSC2_FREQ_R_MAIN -> /OSC2_FREQ_L_MAIN
- J7 pad 9: /OSC2_FILTER_MOD_MAIN -> /OSC2_SIGNAL_MAIN
- Q4 pad 2: Net-(Q4-B) -> /FILTER_FREQ_CV_MAIN
- R27 pad 1: Net-(D5-K) -> GND
- R27 pad 2: Net-(Q2-B) -> Net-(D5-K)
- R46 pad 1: /FILTER_FREQ_CV_MAIN -> Net-(Q2-B)
- R46 pad 2: Net-(Q4-B) -> GND
- R51 pad 1: Net-(Q4-B) -> /FILTER_FREQ_CV_MAIN
- SW1 pad 1: /OSC2_LFO_CAP_CTRL -> /OSC2_LFO_CTRL
- SW1 pad 2: /OSC2_LFO_CTRL -> /OSC2_LFO_CAP_CTRL
Routing:
- net /OSC1_FREQ_L_MAIN: track 33.9 -> 3.53 mm, vias 1 -> 0
- net Net-(C12-Pad2): track 8.80 -> 34.0 mm
- net /RES_AMOUNT_MAIN: track 18.0 -> 40.7 mm
- net /FINAL_OUTPUT_MAIN: track 33.6 -> 18.4 mm
- net -12V: track 452.2 -> 437.3 mm
- net /FILTER_FREQ_CV_MAIN: track 12.4 -> 26.9 mm
- net /OSC2_SIGNAL_MAIN: track 34.5 -> 48.4 mm
- net Net-(Q8-B): track 0.00 -> 11.8 mm
- net Net-(Q4-B): track 11.2 -> 0.00 mm
- net Net-(Q2-B): track 18.9 -> 29.8 mm
- net Net-(Q6-E): track 24.6 -> 14.3 mm
- net Net-(U3A-+): track 27.4 -> 36.2 mm
- net /PIEZO_MAIN: track 11.8 -> 3.78 mm
- net Net-(R12-Pad1): track 23.8 -> 31.8 mm
- net Net-(U4A--): track 16.8 -> 9.00 mm
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Other:
- board text added: "noise volume"
