File: kicad/magnum-drum-synth.kicad_pcb (KiCad board)
At the start: 2 copper layers, 202 x 105 mm, 186 parts, among them J1 Conn_02x10_Odd_Even, J10 Eurorack Mono Jack, J11 Eurorack Mono Jack, J2 Conn_01x04_Socket, J3 locked, J4 Conn_01x03_Header, J5 Conn_01x03_Header, J6 Conn_01x04_Header, J7 Conn_02x10_Odd_Even, J8 Eurorack Mono Jack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

Commit message: rev06 gerbers
Other:
- board text added: "Magnum Percussion Instrument rev 06"
Changed lines of the file:
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@@
   (title_block
     (title "Magnum Percussion Instrument")
-    (date "2022-09-29")
-    (rev "r05")
+    (date "2023-07-19")
+    (rev "r06")
     (comment 2 "creativecommons.org/licenses/by/4.0/")
     (comment 3 "License: CC BY 4.0")
@@
     (effects (font (size 1 1) (thickness 0.15)))
   )
-  (gr_text "Magnum Percussion\nInstrument\nrev 05" (at 138.2 116.2 90) (layer "F.SilkS")
+  (gr_text "Magnum Percussion\nInstrument\nrev 06" (at 138.2 116.2 90) (layer "F.SilkS")
     (effects (font (size 1 1) (thickness 0.15)))
   )

Commit message: Final tweaks
Parts:
- added H13: MountingHole_Pad, Rumblesan_Standard_Parts:MountingHole_3.2mm_M3_DIN965_Pad, F.Cu at (135.2, 33.2)
- added H14: MountingHole_Pad, Rumblesan_Standard_Parts:MountingHole_3.2mm_M3_DIN965_Pad, F.Cu at (33.2, 33.2)
- added H15: MountingHole_Pad, Rumblesan_Standard_Parts:MountingHole_3.2mm_M3_DIN965_Pad, F.Cu at (126.8, 131.8)
- added H16: MountingHole_Pad, Rumblesan_Standard_Parts:MountingHole_3.2mm_M3_DIN965_Pad, F.Cu at (228.8, 131.8)
- Q7: value BC547 -> 2N3904
- Q8: value BC549C -> 2N3904
- R2: value 10k -> 100k
- R25: value 100k -> 10k
- moved R70 7.74 mm to (223.5, 133.1), turned to 90 degrees
- moved D4 6.35 mm to (146.4, 45.1)
- moved J3 6.04 mm to (140.1, 52.8)
- moved Q7 4.89 mm to (219.5, 53.8), turned to 180 degrees
Connections:
- Q7 pad 1: unconnected-(Q7-C-Pad1) -> Net-(Q7-E)
- Q7 pad 3: Net-(Q7-E) -> unconnected-(Q7-C-Pad3)
Routing:
- net Net-(J10-Tip): track 132.1 -> 120.9 mm
- net /Filter/Output: track 36.1 -> 44.3 mm
- net -12V: track 437.3 -> 429.1 mm
- net Net-(D3-A): track 9.39 -> 14.0 mm
- net Net-(Q7-E): track 8.27 -> 7.61 mm
- net /FINAL_OUTPUT_CTRL: track 89.1 -> 88.6 mm, vias 0 -> 1
Other:
- board text added: "Magnum Percussion Instrument rev 06.1"
- board text removed: "Magnum Percussion Instrument rev 06"
